File: LCD_Touchscreen.sch (KiCad schematic (older format))
At the start: 6 parts, among them Con1 52746-0671, Con2 505110-2491

Commit message: Added stm32mp1 module and arduino shield
Parts:
- removed L2: EMI8133MUTAG, Inductors:EMI8133MUTAG, symbol Inductors:EMI8133MUTAG
Connections:
- net labels removed: MIPI_CLK+, MIPI_CLK-, MIPI_D0+, MIPI_D0-, MIPI_D1+, MIPI_D1-
- wire segments 92 -> 82
Changed lines of the file:
@@
 $Descr A3 16535 11693
 encoding utf-8
-Sheet 2 4
+Sheet 2 5
 Title "LCD MiPi and Touchscreen module"
 Date "2020-12-19"
@@
 Wire Wire Line
 	8000 2450 8250 2450
-$Comp
-L Inductors:EMI8133MUTAG L2
-U 1 1 5E8D03CD
-P 7450 5050
-F 0 "L2" H 7450 6365 50  0000 C CNN
-F 1 "EMI8133MUTAG" H 7450 6274 50  0000 C CNN
-F 2 "Inductors:EMI8133MUTAG" H 8900 5100 50  0001 C CNN
-F 3 "https://pl.mouser.com/datasheet/2/308/EMI8132-D-1803782.pdf" H 8900 5100 50  0001 C CNN
-F 4 "ON Semiconductor" H 8150 7500 50  0001 C CNN "Manufacturer"
-F 5 "EMI8133MUTAG" H 8150 7500 50  0001 C CNN "Manufacturer Part Number"
-F 6 "Mouser" H 8150 7500 50  0001 C CNN "Supplier"
-F 7 "863-EMI8133MUTAG" H 8150 7500 50  0001 C CNN "Supplier Part Number"
-F 8 "https://pl.mouser.com/ProductDetail/ON-Semiconductor/EMI8133MUTAG?qs=k6dkFvHqcvCNpFKZjcGIKw%3D%3D" H 8150 7500 50  0001 C CNN "URL"
-F 9 "3,81" H 8200 7500 50  0001 C CNN "Price@10pc"
-F 10 "1,74" H 8200 7500 50  0001 C CNN "Price@500pc"
-F 11 "MW" H 8200 7500 50  0001 C CNN "Developer"
-F 12 "XDFN-16" H 8150 7500 50  0001 C CNN "Package"
-	1    7450 5050
-	-1   0    0    -1
-$EndComp
-$Comp
-L power:GND #PWR0113
-U 1 1 5E96E9DC
-P 6850 6500
-F 0 "#PWR0113" H 6850 6600 30  0001 C CNN
-F 1 "GND" H 6850 6400 30  0001 C CNN
-F 2 "" H 6850 6500 60  0000 C CNN
-F 3 "" H 6850 6500 60  0000 C CNN
-	1    6850 6500
-	1    0    0    -1
-$EndComp
-$Comp
-L power:GND #PWR0114
-U 1 1 5E96E9E6
-P 7050 6500
-F 0 "#PWR0114" H 7050 6600 30  0001 C CNN
-F 1 "GND" H 7050 6400 30  0001 C CNN
-F 2 "" H 7050 6500 60  0000 C CNN
-F 3 "" H 7050 6500 60  0000 C CNN
-	1    7050 6500
-	1    0    0    -1
-$EndComp
-$Comp
-L power:GND #PWR0115
-U 1 1 5E979393
-P 7950 6500
-F 0 "#PWR0115" H 7950 6600 30  0001 C CNN
-F 1 "GND" H 7950 6400 30  0001 C CNN
-F 2 "" H 7950 6500 60  0000 C CNN
-F 3 "" H 7950 6500 60  0000 C CNN
-	1    7950 6500
-	1    0    0    -1
-$EndComp
-$Comp
-L power:GND #PWR0116
-U 1 1 5E97939D
-P 8150 6500
-F 0 "#PWR0116" H 8150 6600 30  0001 C CNN
-F 1 "GND" H 8150 6400 30  0001 C CNN
-F 2 "" H 8150 6500 60  0000 C CNN
-F 3 "" H 8150 6500 60  0000 C CNN
-	1    8150 6500
-	1    0    0    -1
-$EndComp
-Wire Wire Line
-	8150 6400 8150 6500
-Wire Wire Line
-	7950 6400 7950 6500
-Wire Wire Line
-	7050 6400 7050 6500
-Wire Wire Line
-	6850 6400 6850 6500
-Wire Wire Line
-	6200 4000 2400 4000
 Text HLabel 2400 4000 0    50   Input ~ 0
 LCD_MIPI_D0-
-Wire Wire Line
-	6200 4400 2400 4400
 Text HLabel 2400 4400 0    50   Input ~ 0
 LCD_MIPI_D0+
-Wire Wire Line
-	6200 4550 2400 4550
 Text HLabel 2400 4550 0    50   Input ~ 0
 LCD_MIPI_D1-
-Wire Wire Line
-	6200 4950 2400 4950
 Text HLabel 2400 4950 0    50   Input ~ 0
 LCD_MIPI_D1+
-Wire Wire Line
-	6200 5500 2400 5500
 Text HLabel 2400 5500 0    50   Input ~ 0
 LCD_MIPI_CLK+
-Wire Wire Line
-	6200 5100 2400 5100
 Text HLabel 2400 5100 0    50   Input ~ 0
 LCD_MIPI_CLK-
@@
 Wire Wire Line
 	2600 2150 2400 2150
-Text Label 9700 5500 0    50   ~ 0
-MIPI_CLK+
-Text Label 9700 5100 0    50   ~ 0
-MIPI_CLK-
-Text Label 9700 4000 0    50   ~ 0
-MIPI_D0-
-Text Label 9700 4400 0    50   ~ 0
-MIPI_D0+
-Text Label 9700 4550 0    50   ~ 0
-MIPI_D1-
-Text Label 9700 4950 0    50   ~ 0
-MIPI_D1+
 $Comp
 L Inductors:BLM15HG601SN1D L4
@@
 	12550 5650 12550 4000
 Wire Wire Line
-	12550 4000 8700 4000
-Wire Wire Line
-	12450 4400 8700 4400
-Wire Wire Line
 	14450 5550 12450 5550
 Wire Wire Line
@@
 	12350 5350 12350 4550
 Wire Wire Line
-	12350 4550 8700 4550
-Wire Wire Line
 	14450 5250 12250 5250
 Wire Wire Line
 	12250 5250 12250 4950
 Wire Wire Line
-	12250 4950 8700 4950
-Wire Wire Line
 	14450 5050 11800 5050
 Wire Wire Line
 	11800 5050 11800 5100
 Wire Wire Line
-	11800 5100 8700 5100
-Wire Wire Line
 	14450 4950 12650 4950
 Wire Wire Line
 	12650 4950 12650 5500
-Wire Wire Line
-	12650 5500 8700 5500
 $Comp
 L Fpc_Connectors:52746-0671 Con1
@@
 	1    0    0    1
 $EndComp
+Wire Wire Line
+	2400 4000 12550 4000
+Wire Wire Line
+	2400 4400 12450 4400
+Wire Wire Line
+	2400 4550 12350 4550
+Wire Wire Line
+	2400 4950 12250 4950
+Wire Wire Line
+	2400 5100 11800 5100
+Wire Wire Line
+	2400 5500 12650 5500
 $EndSCHEMATC

Commit message: Added Mipi Dsi connection, started stlink module
Connections:
- net LCD_LED+ renamed LCD Backlight Controller/BACKLIGHT_HIGH
- net LCD_LED- renamed LCD Backlight Controller/BACKLIGHT_LOW
Changed lines of the file:
@@
 $Descr A3 16535 11693
 encoding utf-8
-Sheet 2 6
+Sheet 2 8
 Title "LCD MiPi and Touchscreen module"
 Date "2020-12-19"
@@
 F6 "POWER_SUPPLY_2.7-5.5V_GND" I L 6600 2150 50
 $EndSheet
-Wire Wire Line
-	8000 2550 8250 2550
-Wire Wire Line
-	8000 2450 8250 2450
-Text HLabel 2400 4000 0    50   Input ~ 0
+Text HLabel 2400 5650 0    50   Input ~ 0
 LCD_MIPI_D0-
-Text HLabel 2400 4400 0    50   Input ~ 0
+Text HLabel 2400 5550 0    50   Input ~ 0
 LCD_MIPI_D0+
-Text HLabel 2400 4550 0    50   Input ~ 0
+Text HLabel 2400 5350 0    50   Input ~ 0
 LCD_MIPI_D1-
+Text HLabel 2400 5250 0    50   Input ~ 0
+LCD_MIPI_D1+
 Text HLabel 2400 4950 0    50   Input ~ 0
-LCD_MIPI_D1+
-Text HLabel 2400 5500 0    50   Input ~ 0
 LCD_MIPI_CLK+
-Text HLabel 2400 5100 0    50   Input ~ 0
+Text HLabel 2400 5050 0    50   Input ~ 0
 LCD_MIPI_CLK-
 Text HLabel 2250 2900 0    50   Input ~ 0
@@
 Text HLabel 2450 7100 0    50   Input ~ 0
 TP_RESET_1V8
-Text HLabel 2450 7400 0    50   Input ~ 0
+Text HLabel 2450 7400 0    50   Output ~ 0
 TP_NT_1V8
 Text HLabel 2250 1300 0    50   Input ~ 0
@@
 Wire Wire Line
 	6600 2150 2600 2150
-Wire Wire Line
-	8250 2550 8250 3350
-Wire Wire Line
-	8250 3350 2250 3350
-Wire Wire Line
-	8250 2450 8250 1600
-Wire Wire Line
-	8250 1600 2250 1600
-Text HLabel 2250 3350 0    50   Input ~ 0
-LCD_LED+
-Text HLabel 2250 1600 0    50   Input ~ 0
-LCD_LED-
 Wire Wire Line
 	2600 2200 2600 2150
@@
 	14350 4550 14450 4550
 Wire Wire Line
-	8250 2450 14250 2450
-Wire Wire Line
 	14250 2450 14250 3650
 Wire Wire Line
 	14250 3650 14450 3650
-Connection ~ 8250 2450
 Wire Wire Line
 	14450 3750 14150 3750
 Wire Wire Line
 	14150 3750 14150 2550
-Connection ~ 8250 2550
 Wire Wire Line
 	14450 4650 14050 4650
@@
 Wire Wire Line
 	2250 1300 14050 1300
-Wire Wire Line
-	14150 2550 8250 2550
 Wire Wire Line
 	13950 4750 13950 1450
@@
 	1    0    0    -1
 $EndComp
-Wire Wire Line
-	14450 5650 12550 5650
-Wire Wire Line
-	12550 5650 12550 4000
-Wire Wire Line
-	14450 5550 12450 5550
-Wire Wire Line
-	12450 4400 12450 5550
-Wire Wire Line
-	14450 5350 12350 5350
-Wire Wire Line
-	12350 5350 12350 4550
-Wire Wire Line
-	14450 5250 12250 5250
-Wire Wire Line
-	12250 5250 12250 4950
-Wire Wire Line
-	14450 5050 11800 5050
-Wire Wire Line
-	11800 5050 11800 5100
-Wire Wire Line
-	14450 4950 12650 4950
-Wire Wire Line
-	12650 4950 12650 5500
 $Comp
 L Fpc_Connectors:52746-0671 Con1
@@
 $EndComp
 Wire Wire Line
-	2400 4000 12550 4000
-Wire Wire Line
-	2400 4400 12450 4400
-Wire Wire Line
-	2400 4550 12350 4550
-Wire Wire Line
-	2400 4950 12250 4950
-Wire Wire Line
-	2400 5100 11800 5100
-Wire Wire Line
-	2400 5500 12650 5500
+	14450 5650 2400 5650
+Wire Wire Line
+	14450 5550 2400 5550
+Wire Wire Line
+	14450 5250 2400 5250
+Wire Wire Line
+	14450 5050 2400 5050
+Wire Wire Line
+	14450 4950 2400 4950
+Wire Wire Line
+	14450 5350 2400 5350
+Wire Wire Line
+	8000 2550 14150 2550
+Wire Wire Line
+	8000 2450 14250 2450
 $EndSCHEMATC

Commit message: Tracking finished, started tunning
Changed lines of the file:
@@
 Text HLabel 2250 2000 0    50   Input ~ 0
 LCD_VDD_2.7-5.5V
-Wire Wire Line
-	6600 2000 2600 2000
 Text HLabel 2450 7300 0    50   BiDi ~ 0
 TP_SDA_1V8
@@
 	8400 7850 8400 7600
 Wire Wire Line
-	2400 1900 2400 2000
-Connection ~ 2400 2000
-Wire Wire Line
-	2400 2000 2250 2000
-$Comp
-L power:VDD #PWR0108
-U 1 1 5EAB2D4C
-P 2400 1900
-F 0 "#PWR0108" H 2400 2000 30  0001 C CNN
-F 1 "VDD" H 2412 2058 30  0000 C CNN
-F 2 "" H 2400 1900 60  0000 C CNN
-F 3 "" H 2400 1900 60  0000 C CNN
-	1    2400 1900
-	1    0    0    -1
-$EndComp
-$Comp
-L power:VDD #PWR0117
-U 1 1 5EAB31A5
-P 6700 7750
-F 0 "#PWR0117" H 6700 7850 30  0001 C CNN
-F 1 "VDD" V 6700 7900 30  0000 C CNN
-F 2 "" H 6700 7750 60  0000 C CNN
-F 3 "" H 6700 7750 60  0000 C CNN
-	1    6700 7750
-	0    -1   -1   0
-$EndComp
-Wire Wire Line
 	6800 7750 6700 7750
 $Comp
@@
 Wire Wire Line
 	2400 2150 2250 2150
-$Comp
-L power:PWR_FLAG #FLG0101
-U 1 1 5EACCE3D
-P 2600 1950
-F 0 "#FLG0101" H 2600 2220 30  0001 C CNN
-F 1 "PWR_FLAG" H 2600 2208 30  0000 C CNN
-F 2 "" H 2600 1950 60  0000 C CNN
-F 3 "" H 2600 1950 60  0000 C CNN
-	1    2600 1950
-	1    0    0    -1
-$EndComp
-Wire Wire Line
-	2600 1950 2600 2000
-Connection ~ 2600 2000
-Wire Wire Line
-	2600 2000 2400 2000
-$Comp
-L power:PWR_FLAG #FLG0102
-U 1 1 5EAD0960
-P 2600 2200
-F 0 "#FLG0102" H 2600 2470 30  0001 C CNN
-F 1 "PWR_FLAG" H 2600 2458 30  0000 C CNN
-F 2 "" H 2600 2200 60  0000 C CNN
-F 3 "" H 2600 2200 60  0000 C CNN
-	1    2600 2200
-	-1   0    0    1
-$EndComp
-Wire Wire Line
-	6600 2150 2600 2150
-Wire Wire Line
-	2600 2200 2600 2150
-Connection ~ 2600 2150
-Wire Wire Line
-	2600 2150 2400 2150
 $Comp
 L Inductors:BLM15HG601SN1D L4
@@
 Wire Wire Line
 	8000 2450 14250 2450
+Wire Wire Line
+	2400 2150 6600 2150
+Wire Wire Line
+	2250 2000 6600 2000
+Text Label 2600 2000 0    50   ~ 0
+VDD
+Text Label 6700 7750 2    50   ~ 0
+VDD
 $EndSCHEMATC
