File: ethernet.sch (KiCad schematic (older format))
At the start: 42 parts, among them T2 WE-RJ45_74990101210, U7 KSZ8041NL_RNL, X2 ECS-2016MV-250-CN-TR

Commit message: Tracking finished, started tunning
Connections:
- no-connect marks 4 -> 6
Changed lines of the file:
@@
 $Descr A3 16535 11693
 encoding utf-8
-Sheet 10 11
+Sheet 9 11
 Title "Ethernet"
 Date "2021-01-13"
@@
 Wire Wire Line
 	11650 3800 15650 3800
+NoConn ~ 14100 4950
+NoConn ~ 14100 4850
 $EndSCHEMATC
