File: mpu_module.kicad_sch (KiCad schematic)
At the start: 11 parts

Commit message: Started issues implementation
Connections:
- net UART8-CTS renamed PD14-GPIO
- net UART8-RTS renamed PG7-GPIO
- net UART8-RXD renamed PE0-GPIO
- net UART8-TXD renamed PE1-GPIO
Changed lines of the file:
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@@
     (effects (font (size 1.27 1.27)) (justify right))
   )
-  (hierarchical_label "UART8-RTS" (shape output) (at 83.82 238.76 180)
+  (hierarchical_label "PG7-GPIO" (shape output) (at 83.82 238.76 180)
     (effects (font (size 1.27 1.27)) (justify right))
   )
@@
     (effects (font (size 1.27 1.27)) (justify right))
   )
-  (hierarchical_label "UART8-CTS" (shape input) (at 132.08 279.4 180)
+  (hierarchical_label "PD14-GPIO" (shape input) (at 132.08 279.4 180)
     (effects (font (size 1.27 1.27)) (justify right))
   )
@@
     (effects (font (size 1.27 1.27)) (justify right))
   )
-  (hierarchical_label "UART8-RXD" (shape input) (at 238.76 204.47 180)
+  (hierarchical_label "PE0-GPIO" (shape input) (at 238.76 204.47 180)
     (effects (font (size 1.27 1.27)) (justify right))
   )
-  (hierarchical_label "UART8-TXD" (shape output) (at 238.76 208.28 180)
+  (hierarchical_label "PE1-GPIO" (shape output) (at 238.76 208.28 180)
     (effects (font (size 1.27 1.27)) (justify right))
   )

Commit message: Reworked schematic and applied changes on pcb related with mini pci express
Connections:
- net PE0-GPIO renamed PE0-GPIO/UART8_RX
- net PE1-GPIO renamed PE1-GPIO/UART8_TX
Changed lines of the file:
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@@
     (effects (font (size 1.27 1.27)) (justify right))
   )
-  (hierarchical_label "PE0-GPIO" (shape input) (at 238.76 204.47 180)
+  (hierarchical_label "PE0-GPIO{slash}UART8_RX" (shape input) (at 238.76 204.47 180)
     (effects (font (size 1.27 1.27)) (justify right))
   )
-  (hierarchical_label "PE1-GPIO" (shape output) (at 238.76 208.28 180)
+  (hierarchical_label "PE1-GPIO{slash}UART8_TX" (shape output) (at 238.76 208.28 180)
     (effects (font (size 1.27 1.27)) (justify right))
   )
@@
     (pin "2")
   )
-  (symbol (lib_id "VisionSOM:VisionSOM-STM32MP1") (at 58.42 271.78 0) (unit 10)
+  (symbol (lib_name "VisionSOM:VisionSOM-STM32MP1_9") (lib_id "VisionSOM:VisionSOM-STM32MP1") (at 58.42 271.78 0) (unit 10)
     (in_bom yes) (on_board yes)
     (property "Reference" "SOM1" (id 0) (at 55.88 259.08 0)
@@
     (pin "27")
   )
-  (symbol (lib_id "VisionSOM:VisionSOM-STM32MP1") (at 86.36 189.23 0) (unit 2)
+  (symbol (lib_name "VisionSOM:VisionSOM-STM32MP1_8") (lib_id "VisionSOM:VisionSOM-STM32MP1") (at 86.36 189.23 0) (unit 2)
     (in_bom yes) (on_board yes)
     (property "Reference" "SOM1" (id 0) (at 115.0112 188.0616 0)
@@
     (pin "9")
   )
-  (symbol (lib_id "VisionSOM:VisionSOM-STM32MP1") (at 219.71 269.24 0) (unit 7)
+  (symbol (lib_name "VisionSOM:VisionSOM-STM32MP1_2") (lib_id "VisionSOM:VisionSOM-STM32MP1") (at 219.71 269.24 0) (unit 7)
     (in_bom yes) (on_board yes)
     (property "Reference" "SOM1" (id 0) (at 273.05 252.73 0))
@@
     (pin "78")
   )
-  (symbol (lib_id "VisionSOM:VisionSOM-STM32MP1") (at 186.69 238.76 0) (unit 9)
+  (symbol (lib_name "VisionSOM:VisionSOM-STM32MP1_3") (lib_id "VisionSOM:VisionSOM-STM32MP1") (at 186.69 238.76 0) (unit 9)
     (in_bom yes) (on_board yes)
     (property "Reference" "SOM1" (id 0) (at 166.37 220.98 0))
@@
     (pin "79")
   )
-  (symbol (lib_id "VisionSOM:VisionSOM-STM32MP1") (at 323.85 204.47 0) (unit 8)
+  (symbol (lib_name "VisionSOM:VisionSOM-STM32MP1_7") (lib_id "VisionSOM:VisionSOM-STM32MP1") (at 323.85 204.47 0) (unit 8)
     (in_bom yes) (on_board yes)
     (property "Reference" "SOM1" (id 0) (at 364.49 224.79 0))
@@
     (pin "63")
   )
-  (symbol (lib_id "VisionSOM:VisionSOM-STM32MP1") (at 298.45 165.1 0) (unit 6)
+  (symbol (lib_name "VisionSOM:VisionSOM-STM32MP1_6") (lib_id "VisionSOM:VisionSOM-STM32MP1") (at 298.45 165.1 0) (unit 6)
     (in_bom yes) (on_board yes)
     (property "Reference" "SOM1" (id 0) (at 308.9148 143.129 0))
@@
     (pin "99")
   )
-  (symbol (lib_id "VisionSOM:VisionSOM-STM32MP1") (at 86.36 91.44 0) (unit 1)
+  (symbol (lib_name "VisionSOM:VisionSOM-STM32MP1_1") (lib_id "VisionSOM:VisionSOM-STM32MP1") (at 86.36 91.44 0) (unit 1)
     (in_bom yes) (on_board yes)
     (property "Reference" "SOM1" (id 0) (at 86.36 14.859 0))
@@
     (pin "41")
     (pin "42")
-    (pin "43")
     (pin "44")
     (pin "50")
@@
     (pin "98")
   )
-  (symbol (lib_id "VisionSOM:VisionSOM-STM32MP1") (at 285.75 111.76 0) (unit 5)
+  (symbol (lib_name "VisionSOM:VisionSOM-STM32MP1_5") (lib_id "VisionSOM:VisionSOM-STM32MP1") (at 285.75 111.76 0) (unit 5)
     (in_bom yes) (on_board yes)
     (property "Reference" "SOM1" (id 0) (at 298.1198 78.359 0))
@@
     (pin "77")
   )
-  (symbol (lib_id "VisionSOM:VisionSOM-STM32MP1") (at 275.59 46.99 0) (unit 4)
+  (symbol (lib_name "VisionSOM:VisionSOM-STM32MP1_4") (lib_id "VisionSOM:VisionSOM-STM32MP1") (at 275.59 46.99 0) (unit 4)
     (in_bom yes) (on_board yes)
     (property "Reference" "SOM1" (id 0) (at 291.7698 13.589 0))
