File: mpu_module.kicad_sch (KiCad schematic)
At the start: 11 parts

Commit message: Updated schematic and pdf
Connections:
- net PG13-GPIO is gone; now on net ENET1-TXD0: SOM1.122 (PG13_TRACED0,LPTIM1_OUT,SAI1_CK2,SAI4_CK1,SPI6_SCK,SAI1_SCK_A,USART6_CTS/USART6_NSS,SAI4_MCLK_A,ETH1_GMII_TXD0/ETH1_MII_TXD0/ETH1_RGMII_TXD0/ETH1_RMII_TXD0,FMC_A24,LCD_R0,EVENTOUT)
- net ENET1-TXD0: no longer SOM1.79 (PG14_TRACED1,LPTIM1_ETR,SPI6_MOSI,_SAI4_D1,USART6_TX,QUADSPI_BK2_IO3,SAI4_SD_A,ETH1_GMII_TXD1/ETH1_MII_TXD1/ETH1_RGMII_TXD1/ETH1_RMII_TXD1,FMC_A25,LCD_B0,EVENTOUT)
- new net PG14-GPIO: SOM1.79 (PG14_TRACED1,LPTIM1_ETR,SPI6_MOSI,_SAI4_D1,USART6_TX,QUADSPI_BK2_IO3,SAI4_SD_A,ETH1_GMII_TXD1/ETH1_MII_TXD1/ETH1_RGMII_TXD1/ETH1_RMII_TXD1,FMC_A25,LCD_B0,EVENTOUT)

Commit message: Modified ethernet
Connections:
- net ADC1_INP13 renamed ENET1-TX-CLK
- net ADC1_INP15 renamed ENET1-COL
- net ENET1-CRS-DV renamed ENET1-RX-DV
- net ENET1-REFCLK renamed ENET1-RX-CLK
- net PA0-GPIO renamed ENET1-CRS
Changed lines of the file:
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@@
     (effects (font (size 1.27 1.27)) (justify right))
   )
-  (hierarchical_label "ENET1-CRS-DV" (shape bidirectional) (at 142.24 24.13 180)
+  (hierarchical_label "ENET1-RX-DV" (shape output) (at 142.24 24.13 180)
     (effects (font (size 1.27 1.27)) (justify right))
   )
-  (hierarchical_label "ENET1-REFCLK" (shape bidirectional) (at 142.24 27.94 180)
+  (hierarchical_label "ENET1-RX-CLK" (shape output) (at 142.24 27.94 180)
     (effects (font (size 1.27 1.27)) (justify right))
   )
-  (hierarchical_label "ADC1_INP15" (shape input) (at 142.24 31.75 180)
+  (hierarchical_label "ENET1-COL" (shape output) (at 142.24 31.75 180)
     (effects (font (size 1.27 1.27)) (justify right))
   )
@@
     (effects (font (size 1.27 1.27)) (justify right))
   )
-  (hierarchical_label "PA0-GPIO" (shape bidirectional) (at 142.24 73.66 180)
+  (hierarchical_label "ENET1-CRS" (shape output) (at 142.24 73.66 180)
     (effects (font (size 1.27 1.27)) (justify right))
   )
@@
     (effects (font (size 1.27 1.27)) (justify right))
   )
-  (hierarchical_label "ENET1-MDC" (shape bidirectional) (at 187.96 172.72 180)
+  (hierarchical_label "ENET1-MDC" (shape output) (at 187.96 172.72 180)
     (effects (font (size 1.27 1.27)) (justify right))
   )
-  (hierarchical_label "ADC1_INP13" (shape input) (at 187.96 176.53 180)
+  (hierarchical_label "ENET1-TX-CLK" (shape output) (at 187.96 176.53 180)
     (effects (font (size 1.27 1.27)) (justify right))
   )

Commit message: Updated schematic
Connections:
- net JTAG-~TRST~ renamed JTAG-~{TRST}
- net STM32-~RST~ renamed STM32-~{RST}
