File: LCD_Backlight_Driver.kicad_sch (KiCad schematic)
At the start: 6 parts, among them U1 TPS61169DCKR

Commit message: Reworked schematic and applied changes on pcb related with mini pci express
Parts:
- removed R1: 10R/1%/0.1Wat, Resistor_Smd_0603:10R_0603, symbol Resistors_Smd0603:10R_0603_1%
- added R1: 10Ω/1%/0.1Wat, Resistor_Smd_0603:10R_0603, symbol Resistors_Smd0603:10R_1%
Connections:
- net BACKLIGHT_LOW: now also R1.1
- net GND: now also R1.2
Changed lines of the file:
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@@
     (pin "1")
   )
-  (symbol (lib_id "Resistors_Smd0603:10R_0603_1%") (at 226.06 139.7 0) (unit 1)
+  (symbol (lib_id "Resistors_Smd0603:10R_1%") (at 226.06 139.7 0) (unit 1)
     (in_bom yes) (on_board yes)
-    (property "Reference" "R1" (id 0) (at 227.7872 138.5316 0)
+    (property "Reference" "R1" (id 0) (at 227.711 138.551 0)
       (effects (font (size 1.27 1.27)) (justify left))
     )
-    (property "Value" "10R/1%/0.1Wat" (id 1) (at 227.7872 140.843 0)
+    (property "Value" "10Ω/1%/0.1Wat" (id 1) (at 227.711 140.849 0)
       (effects (font (size 1.27 1.27)) (justify left))
     )
@@
       (effects (font (size 1.27 1.27)) hide)
     )
-    (property "Package" "0603" (id 11) (at 226.06 139.7 0)
+    (property "Developer" "MW" (id 11) (at 226.06 139.7 0)
       (effects (font (size 1.27 1.27)) hide)
     )
-    (property "Developer" "MW" (id 12) (at 226.06 139.7 0)
+    (property "Package" "0603" (id 12) (at 226.06 139.7 0)
       (effects (font (size 1.27 1.27)) hide)
     )
