File: LCD_Backlight_Driver.kicad_sch (KiCad schematic)
At the start: 6 parts, among them U1 TPS61169DCKR

Commit message: Cleared all errors DRC
Parts:
- C1: symbol Capacitors_Smd0603:1uF_0603 -> Capacitors_Smd0603:1uF; LCSC Part #(optional) (none) -> C105504
Changed lines of the file:
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@@
     (pin "5")
   )
-  (symbol (lib_id "Capacitors_Smd0603:1uF_0603") (at 184.15 113.03 0) (unit 1)
+  (symbol (lib_id "Capacitors_Smd0603:1uF") (at 184.15 113.03 0) (unit 1)
     (in_bom yes) (on_board yes)
     (property "Reference" "C1" (id 0) (at 187.4774 111.8616 0)
@@
       (effects (font (size 1.524 1.524)) hide)
     )
-    (property "Datasheet" "Capacitors/Smd_0603/Components_Documentation/KEM_C1005_Y5V_SMD.pdf" (id 3) (at 180.34 107.95 0)
+    (property "Datasheet" "https://www.tme.eu/Document/4a42202b32dab16128fe107dd69598cc/samsung-chip-cap.pdf" (id 3) (at 180.34 107.95 0)
       (effects (font (size 1.524 1.524)) hide)
     )
@@
       (effects (font (size 1.27 1.27)) hide)
     )
+    (property "LCSC Part #(optional)" "C105504" (id 12) (at 184.15 113.03 0)
+      (effects (font (size 1.27 1.27)) hide)
+    )

Commit message: Gerbers created, BOM, CPL
Parts:
- C1: value 1uF/6V3 -> 1uF/16V
Changed lines of the file:
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@@
     (pin "5")
-  )
-  (symbol (lib_id "Capacitors_Smd0603:1uF") (at 184.15 113.03 0) (unit 1)
-    (in_bom yes) (on_board yes)
-    (property "Reference" "C1" (id 0) (at 187.4774 111.8616 0)
-      (effects (font (size 1.27 1.27)) (justify left))
-    )
-    (property "Value" "1uF/6V3" (id 1) (at 187.4774 114.173 0)
-      (effects (font (size 1.27 1.27)) (justify left))
-    )
-    (property "Footprint" "Capacitors_Smd_0603:1uF_0603" (id 2) (at 180.34 107.95 0)
-      (effects (font (size 1.524 1.524)) hide)
-    )
-    (property "Datasheet" "https://www.tme.eu/Document/4a42202b32dab16128fe107dd69598cc/samsung-chip-cap.pdf" (id 3) (at 180.34 107.95 0)
-      (effects (font (size 1.524 1.524)) hide)
-    )
-    (property "Manufacturer" "SAMSUNG" (id 4) (at 184.15 113.03 0)
-      (effects (font (size 1.27 1.27)) hide)
-    )
-    (property "Manufacturer Part Number" "CL10B105KO8NNNC" (id 5) (at 184.15 113.03 0)
-      (effects (font (size 1.27 1.27)) hide)
-    )
-    (property "Supplier" "TME" (id 6) (at 184.15 113.03 0)
-      (effects (font (size 1.27 1.27)) hide)
-    )
-    (property "Supplier Part Number" "CL10B105KO8NNNC" (id 7) (at 184.15 113.03 0)
-      (effects (font (size 1.27 1.27)) hide)
-    )
-    (property "URL" "https://www.tme.eu/pl/details/cl10b105ko8nnnc/kondensatory-mlcc-smd-0603/samsung/" (id 8) (at 184.15 113.03 0)
-      (effects (font (size 1.27 1.27)) hide)
-    )
-    (property "Price@1pc" "0,07530" (id 9) (at 184.15 113.03 0)
-      (effects (font (size 1.27 1.27)) hide)
-    )
-    (property "Price@1000pcs" "0,03514" (id 10) (at 184.15 113.03 0)
-      (effects (font (size 1.27 1.27)) hide)
-    )
-    (property "Package" "0603" (id 11) (at 184.15 113.03 0)
-      (effects (font (size 1.27 1.27)) hide)
-    )
-    (property "LCSC Part #(optional)" "C105504" (id 12) (at 184.15 113.03 0)
-      (effects (font (size 1.27 1.27)) hide)
-    )
-    (pin "1")
-    (pin "2")
   )
   (symbol (lib_id "Capacitors_Smd0603:4_7uF_0603") (at 241.3 113.03 0) (unit 1)
@@
     (pin "2")
   )
+  (symbol (lib_id "Capacitors_Smd0603:1uF") (at 184.15 113.03 0) (unit 1)
+    (in_bom yes) (on_board yes) (fields_autoplaced)
+    (property "Reference" "C1" (id 0) (at 180.8226 112.1215 0)
+      (effects (font (size 1.27 1.27)) (justify right))
+    )
+    (property "Value" "1uF/16V" (id 1) (at 180.8226 114.8966 0)
+      (effects (font (size 1.27 1.27)) (justify right))
+    )
+    (property "Footprint" "Capacitors_Smd_0603:1uF_0603" (id 2) (at 180.34 107.95 0)
+      (effects (font (size 1.524 1.524)) hide)
+    )
+    (property "Datasheet" "https://www.tme.eu/Document/4a42202b32dab16128fe107dd69598cc/samsung-chip-cap.pdf" (id 3) (at 180.34 107.95 0)
+      (effects (font (size 1.524 1.524)) hide)
+    )
+    (property "Manufacturer" "SAMSUNG" (id 4) (at 184.15 113.03 0)
+      (effects (font (size 1.27 1.27)) hide)
+    )
+    (property "Manufacturer Part Number" "CL10B105KO8NNNC" (id 5) (at 184.15 113.03 0)
+      (effects (font (size 1.27 1.27)) hide)
+    )
+    (property "Supplier" "TME" (id 6) (at 184.15 113.03 0)
+      (effects (font (size 1.27 1.27)) hide)
+    )
+    (property "Supplier Part Number" "CL10B105KO8NNNC" (id 7) (at 184.15 113.03 0)
+      (effects (font (size 1.27 1.27)) hide)
+    )
+    (property "URL" "https://www.tme.eu/pl/details/cl10b105ko8nnnc/kondensatory-mlcc-smd-0603/samsung/" (id 8) (at 184.15 113.03 0)
+      (effects (font (size 1.27 1.27)) hide)
+    )
+    (property "Price@1pc" "0,07530" (id 9) (at 184.15 113.03 0)
+      (effects (font (size 1.27 1.27)) hide)
+    )
+    (property "Price@1000pcs" "0,03514" (id 10) (at 184.15 113.03 0)
+      (effects (font (size 1.27 1.27)) hide)
+    )
+    (property "Package" "0603" (id 11) (at 184.15 113.03 0)
+      (effects (font (size 1.27 1.27)) hide)
+    )
+    (property "LCSC Part #(optional)" "C105504" (id 12) (at 184.15 113.03 0)
+      (effects (font (size 1.27 1.27)) hide)
+    )
+    (pin "1")
+    (pin "2")
+  )
   (symbol (lib_id "Resistors_Smd0603:10R_1%") (at 226.06 139.7 0) (unit 1)
     (in_bom yes) (on_board yes)
@@
       (effects (font (size 1.27 1.27)) hide)
     )
-    (property "Datasheet" "Resistors/Smd_0603/Components_Documentation/Panasonic_Precision_Resistors_SMD.pdf" (id 3) (at 232.41 147.32 0)
-      (effects (font (size 1.27 1.27)) hide)
-    )
+    (property "Datasheet" "https://www.tme.eu/Document/b315665a56acbc42df513c99b390ad98/ROYALOHM-THICKFILM.pdf" (id 3) (at 232.41 147.32 0)
+      (effects (font (size 1.27 1.27)) hide)
+    )
