File: LCD_Touchscreen.kicad_sch (KiCad schematic)
At the start: 5 parts, among them Con1 52746-0671, Con2 505110-2491

Commit message: Reworked schematic and applied changes on pcb related with mini pci express
Parts:
- C5, C6: symbol Capacitors_Smd0603:100nF_0603 -> Capacitors_Smd0603:100n
Changed lines of the file:
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@@
     (pin "2")
   )
-  (symbol (lib_id "Capacitors_Smd0603:100nF_0603") (at 339.09 213.36 0) (unit 1)
+  (symbol (lib_id "Capacitors_Smd0603:100n") (at 339.09 213.36 0) (unit 1)
     (in_bom yes) (on_board yes)
     (property "Reference" "C5" (id 0) (at 342.4174 212.1916 0)
@@
     (pin "2")
   )
-  (symbol (lib_id "Capacitors_Smd0603:100nF_0603") (at 354.33 185.42 0) (unit 1)
+  (symbol (lib_id "Capacitors_Smd0603:100n") (at 354.33 185.42 0) (unit 1)
     (in_bom yes) (on_board yes)
     (property "Reference" "C6" (id 0) (at 349.25 182.88 0)

Commit message: Applied all changes, tunnign started
Parts:
- added TP10, TP11, TP5, TP6, TP7, TP8, TP9: TP1.27mm, Test_Points:Test_Point_1.27mm, symbol Test_Points:Test_Point_1.27mm
Connections:
- net LCD_BACKLIGHT_PWM: now also TP9.1 (TP)
- net LCD_MIPI_CLK+: now also TP5.1 (TP)
- net LCD_MIPI_CLK-: now also TP6.1 (TP)
- net LCD_MIPI_D0+: now also TP10.1 (TP)
- net LCD_MIPI_D0-: now also TP11.1 (TP)
- net LCD_MIPI_D1+: now also TP7.1 (TP)
- net LCD_MIPI_D1-: now also TP8.1 (TP)
Changed lines of the file:
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@@
   )
   (junction (at 60.96 54.61) (diameter 1.016) (color 0 0 0 0))
+  (junction (at 99.06 125.73) (diameter 1.016) (color 0 0 0 0))
+  (junction (at 111.76 128.27) (diameter 1.016) (color 0 0 0 0))
+  (junction (at 125.73 133.35) (diameter 1.016) (color 0 0 0 0))
+  (junction (at 138.43 135.89) (diameter 1.016) (color 0 0 0 0))
+  (junction (at 146.05 73.66) (diameter 1.016) (color 0 0 0 0))
+  (junction (at 151.13 140.97) (diameter 1.016) (color 0 0 0 0))
+  (junction (at 163.83 143.51) (diameter 1.016) (color 0 0 0 0))
   (junction (at 267.97 190.5) (diameter 1.016) (color 0 0 0 0))
   (junction (at 339.09 199.39) (diameter 1.016) (color 0 0 0 0))
@@
     (stroke (width 0) (type solid) (color 0 0 0 0))
   )
-  (wire (pts (xy 167.64 73.66) (xy 57.15 73.66))
+  (wire (pts (xy 99.06 121.92) (xy 99.06 125.73))
+    (stroke (width 0) (type solid) (color 0 0 0 0))
+  )
+  (wire (pts (xy 99.06 125.73) (xy 60.96 125.73))
+    (stroke (width 0) (type solid) (color 0 0 0 0))
+  )
+  (wire (pts (xy 111.76 121.92) (xy 111.76 128.27))
+    (stroke (width 0) (type solid) (color 0 0 0 0))
+  )
+  (wire (pts (xy 111.76 128.27) (xy 60.96 128.27))
+    (stroke (width 0) (type solid) (color 0 0 0 0))
+  )
+  (wire (pts (xy 125.73 121.92) (xy 125.73 133.35))
+    (stroke (width 0) (type solid) (color 0 0 0 0))
+  )
+  (wire (pts (xy 125.73 133.35) (xy 60.96 133.35))
+    (stroke (width 0) (type solid) (color 0 0 0 0))
+  )
+  (wire (pts (xy 138.43 121.92) (xy 138.43 135.89))
+    (stroke (width 0) (type solid) (color 0 0 0 0))
+  )
+  (wire (pts (xy 138.43 135.89) (xy 60.96 135.89))
+    (stroke (width 0) (type solid) (color 0 0 0 0))
+  )
+  (wire (pts (xy 146.05 71.12) (xy 146.05 73.66))
+    (stroke (width 0) (type solid) (color 0 0 0 0))
+  )
+  (wire (pts (xy 146.05 73.66) (xy 57.15 73.66))
+    (stroke (width 0) (type solid) (color 0 0 0 0))
+  )
+  (wire (pts (xy 151.13 121.92) (xy 151.13 140.97))
+    (stroke (width 0) (type solid) (color 0 0 0 0))
+  )
+  (wire (pts (xy 151.13 140.97) (xy 60.96 140.97))
+    (stroke (width 0) (type solid) (color 0 0 0 0))
+  )
+  (wire (pts (xy 163.83 121.92) (xy 163.83 143.51))
+    (stroke (width 0) (type solid) (color 0 0 0 0))
+  )
+  (wire (pts (xy 163.83 143.51) (xy 60.96 143.51))
+    (stroke (width 0) (type solid) (color 0 0 0 0))
+  )
+  (wire (pts (xy 167.64 73.66) (xy 146.05 73.66))
     (stroke (width 0) (type solid) (color 0 0 0 0))
   )
@@
     (stroke (width 0) (type solid) (color 0 0 0 0))
   )
-  (wire (pts (xy 367.03 125.73) (xy 60.96 125.73))
-    (stroke (width 0) (type solid) (color 0 0 0 0))
-  )
-  (wire (pts (xy 367.03 128.27) (xy 60.96 128.27))
-    (stroke (width 0) (type solid) (color 0 0 0 0))
-  )
-  (wire (pts (xy 367.03 133.35) (xy 60.96 133.35))
-    (stroke (width 0) (type solid) (color 0 0 0 0))
-  )
-  (wire (pts (xy 367.03 135.89) (xy 60.96 135.89))
-    (stroke (width 0) (type solid) (color 0 0 0 0))
-  )
-  (wire (pts (xy 367.03 140.97) (xy 60.96 140.97))
-    (stroke (width 0) (type solid) (color 0 0 0 0))
-  )
-  (wire (pts (xy 367.03 143.51) (xy 60.96 143.51))
+  (wire (pts (xy 367.03 125.73) (xy 99.06 125.73))
+    (stroke (width 0) (type solid) (color 0 0 0 0))
+  )
+  (wire (pts (xy 367.03 128.27) (xy 111.76 128.27))
+    (stroke (width 0) (type solid) (color 0 0 0 0))
+  )
+  (wire (pts (xy 367.03 133.35) (xy 125.73 133.35))
+    (stroke (width 0) (type solid) (color 0 0 0 0))
+  )
+  (wire (pts (xy 367.03 135.89) (xy 138.43 135.89))
+    (stroke (width 0) (type solid) (color 0 0 0 0))
+  )
+  (wire (pts (xy 367.03 140.97) (xy 151.13 140.97))
+    (stroke (width 0) (type solid) (color 0 0 0 0))
+  )
+  (wire (pts (xy 367.03 143.51) (xy 163.83 143.51))
     (stroke (width 0) (type solid) (color 0 0 0 0))
   )
@@
     (pin "2")
   )
+  (symbol (lib_id "Test_Points:Test_Point_1.27mm") (at 99.06 115.57 270) (unit 1)
+    (in_bom yes) (on_board yes) (fields_autoplaced)
+    (property "Reference" "TP5" (id 0) (at 100.9651 117.5396 90)
+      (effects (font (size 1.27 1.27)) (justify left))
+    )
+    (property "Value" "TP1.27mm" (id 1) (at 100.9651 119.8383 90)
+      (effects (font (size 1.27 1.27)) (justify left))
+    )
+    (property "Footprint" "Test_Points:Test_Point_1.27mm" (id 2) (at 105.41 119.38 0)
+      (effects (font (size 1.27 1.27)) hide)
+    )
+    (property "Datasheet" "" (id 3) (at 105.41 119.38 0)
+      (effects (font (size 1.27 1.27)) hide)
+    )
+    (pin "1")
+  )
+  (symbol (lib_id "Test_Points:Test_Point_1.27mm") (at 111.76 115.57 270) (unit 1)
+    (in_bom yes) (on_board yes) (fields_autoplaced)
+    (property "Reference" "TP6" (id 0) (at 113.6651 117.5396 90)
+      (effects (font (size 1.27 1.27)) (justify left))
+    )
+    (property "Value" "TP1.27mm" (id 1) (at 113.6651 119.8383 90)
+      (effects (font (size 1.27 1.27)) (justify left))
+    )
+    (property "Footprint" "Test_Points:Test_Point_1.27mm" (id 2) (at 118.11 119.38 0)
+      (effects (font (size 1.27 1.27)) hide)
+    )
+    (property "Datasheet" "" (id 3) (at 118.11 119.38 0)
+      (effects (font (size 1.27 1.27)) hide)
+    )
+    (pin "1")
+  )
+  (symbol (lib_id "Test_Points:Test_Point_1.27mm") (at 125.73 115.57 270) (unit 1)
+    (in_bom yes) (on_board yes) (fields_autoplaced)
+    (property "Reference" "TP7" (id 0) (at 127.6351 117.5396 90)
+      (effects (font (size 1.27 1.27)) (justify left))
+    )
+    (property "Value" "TP1.27mm" (id 1) (at 127.6351 119.8383 90)
+      (effects (font (size 1.27 1.27)) (justify left))
+    )
+    (property "Footprint" "Test_Points:Test_Point_1.27mm" (id 2) (at 132.08 119.38 0)
+      (effects (font (size 1.27 1.27)) hide)
+    )
+    (property "Datasheet" "" (id 3) (at 132.08 119.38 0)
+      (effects (font (size 1.27 1.27)) hide)
+    )
+    (pin "1")
+  )
+  (symbol (lib_id "Test_Points:Test_Point_1.27mm") (at 138.43 115.57 270) (unit 1)
+    (in_bom yes) (on_board yes) (fields_autoplaced)
+    (property "Reference" "TP8" (id 0) (at 140.3351 117.5396 90)
+      (effects (font (size 1.27 1.27)) (justify left))
+    )
+    (property "Value" "TP1.27mm" (id 1) (at 140.3351 119.8383 90)
+      (effects (font (size 1.27 1.27)) (justify left))
+    )
+    (property "Footprint" "Test_Points:Test_Point_1.27mm" (id 2) (at 144.78 119.38 0)
+      (effects (font (size 1.27 1.27)) hide)
+    )
+    (property "Datasheet" "" (id 3) (at 144.78 119.38 0)
+      (effects (font (size 1.27 1.27)) hide)
+    )
+    (pin "1")
+  )
+  (symbol (lib_id "Test_Points:Test_Point_1.27mm") (at 146.05 64.77 270) (unit 1)
+    (in_bom yes) (on_board yes) (fields_autoplaced)
+    (property "Reference" "TP9" (id 0) (at 147.9551 66.7396 90)
+      (effects (font (size 1.27 1.27)) (justify left))
+    )
+    (property "Value" "TP1.27mm" (id 1) (at 147.9551 69.0383 90)
+      (effects (font (size 1.27 1.27)) (justify left))
+    )
+    (property "Footprint" "Test_Points:Test_Point_1.27mm" (id 2) (at 152.4 68.58 0)
+      (effects (font (size 1.27 1.27)) hide)
+    )
+    (property "Datasheet" "" (id 3) (at 152.4 68.58 0)
+      (effects (font (size 1.27 1.27)) hide)
+    )
+    (pin "1")
+  )
+  (symbol (lib_id "Test_Points:Test_Point_1.27mm") (at 151.13 115.57 270) (unit 1)
+    (in_bom yes) (on_board yes) (fields_autoplaced)
+    (property "Reference" "TP10" (id 0) (at 153.0351 117.5396 90)
+      (effects (font (size 1.27 1.27)) (justify left))
+    )
+    (property "Value" "TP1.27mm" (id 1) (at 153.0351 119.8383 90)
+      (effects (font (size 1.27 1.27)) (justify left))
+    )
+    (property "Footprint" "Test_Points:Test_Point_1.27mm" (id 2) (at 157.48 119.38 0)
+      (effects (font (size 1.27 1.27)) hide)
+    )
+    (property "Datasheet" "" (id 3) (at 157.48 119.38 0)
+      (effects (font (size 1.27 1.27)) hide)
+    )
+    (pin "1")
+  )
+  (symbol (lib_id "Test_Points:Test_Point_1.27mm") (at 163.83 115.57 270) (unit 1)
+    (in_bom yes) (on_board yes) (fields_autoplaced)
+    (property "Reference" "TP11" (id 0) (at 165.7351 117.5396 90)
+      (effects (font (size 1.27 1.27)) (justify left))
+    )
+    (property "Value" "TP1.27mm" (id 1) (at 165.7351 119.8383 90)
+      (effects (font (size 1.27 1.27)) (justify left))
+    )
+    (property "Footprint" "Test_Points:Test_Point_1.27mm" (id 2) (at 170.18 119.38 0)
+      (effects (font (size 1.27 1.27)) hide)
+    )
+    (property "Datasheet" "" (id 3) (at 170.18 119.38 0)
+      (effects (font (size 1.27 1.27)) hide)
+    )
+    (pin "1")
+  )
   (symbol (lib_id "Capacitors_Smd0603:100n") (at 339.09 213.36 0) (unit 1)
