File: LCD_Touchscreen.kicad_sch (KiCad schematic)
At the start: 12 parts, among them Con1 52746-0671, Con2 505110-2491

Commit message: Corrected schematic
Parts:
- renumbered Con1 to CON1, Con2 to CON2
Changed lines of the file:
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@@
   (symbol (lib_id "Fpc_Connectors:24pin_505110-2491_0.5mm") (at 373.38 119.38 0) (unit 1)
     (in_bom yes) (on_board yes)
-    (property "Reference" "Con2" (id 0) (at 380.4412 118.0846 0)
+    (property "Reference" "CON2" (id 0) (at 380.4412 118.0846 0)
       (effects (font (size 1.27 1.27)) (justify left))
     )
@@
   (symbol (lib_id "Fpc_Connectors:52746-0671") (at 278.13 186.69 0) (mirror x) (unit 1)
     (in_bom yes) (on_board yes)
-    (property "Reference" "Con1" (id 0) (at 283.9212 187.7314 0)
+    (property "Reference" "CON1" (id 0) (at 283.9212 187.7314 0)
       (effects (font (size 1.27 1.27)) (justify left))
     )

Commit message: Cleared all errors DRC
Parts:
- L4: Developer (none) -> MW; LCSC Part #(optional) (none) -> C76890; Manufacturer (none) -> MURATA; Manufacturer Part Number (none) -> BLM15HG601SN1D; Package (none) -> 0402; Price@1000pcs (none) -> 0,084; Price@1pc (none) -> 0,248; Supplier (none) -> Tme; Supplier Part Number (none) -> BLM15HG601SN1D; URL (none) -> https://www.tme.eu/pl/details/blm15hg601sn1d/ferryty-korali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
Connections:
- net GND: now also CON1.0 (MNT), CON2.0 (PADS)
Changed lines of the file:
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@@
     (stroke (width 0) (type solid) (color 0 0 0 0))
+  )
+  (wire (pts (xy 280.67 170.815) (xy 280.67 172.72))
+    (stroke (width 0) (type default) (color 0 0 0 0))
   )
   (wire (pts (xy 364.49 123.19) (xy 367.03 123.19))
@@
     (stroke (width 0) (type solid) (color 0 0 0 0))
   )
+  (wire (pts (xy 284.48 170.815) (xy 284.48 175.26))
+    (stroke (width 0) (type solid) (color 0 0 0 0))
+  )
   (wire (pts (xy 354.33 180.34) (xy 354.33 175.26))
     (stroke (width 0) (type solid) (color 0 0 0 0))
@@
   )
   (wire (pts (xy 354.33 175.26) (xy 351.79 175.26))
+    (stroke (width 0) (type solid) (color 0 0 0 0))
+  )
+  (wire (pts (xy 284.48 170.815) (xy 280.67 170.815))
+    (stroke (width 0) (type default) (color 0 0 0 0))
+  )
+  (wire (pts (xy 364.49 151.13) (xy 367.03 151.13))
     (stroke (width 0) (type solid) (color 0 0 0 0))
   )
@@
       (effects (font (size 7.62 7.62)) hide)
     )
-    (property "Datasheet" "C:/Wiktor/KiCad/KiCadWolowik/Schematic/Inductors/Components_Documentation/BLM15HG601SN1#.pdf" (id 3) (at 331.47 162.56 0)
+    (property "Datasheet" "https://www.tme.eu/Document/ea442a092e4ff19cd70ec3627ff4728b/BLM15HG601SN1%23.pdf" (id 3) (at 331.47 162.56 0)
       (effects (font (size 7.62 7.62)) hide)
+    )
+    (property "Manufacturer" "MURATA" (id 4) (at 346.71 175.26 0)
+      (effects (font (size 1.27 1.27)) hide)
+    )
+    (property "Manufacturer Part Number" "BLM15HG601SN1D" (id 5) (at 346.71 175.26 0)
+      (effects (font (size 1.27 1.27)) hide)
+    )
+    (property "Supplier" "Tme" (id 6) (at 346.71 175.26 0)
+      (effects (font (size 1.27 1.27)) hide)
+    )
+    (property "Supplier Part Number" "BLM15HG601SN1D " (id 7) (at 346.71 175.26 0)
+      (effects (font (size 1.27 1.27)) hide)
+    )
+    (property "URL" "https://www.tme.eu/pl/details/blm15hg601sn1d/ferryty-koraliki/murata/" (id 8) (at 346.71 175.26 0)
+      (effects (font (size 1.27 1.27)) hide)
+    )
+    (property "Price@1pc" "0,248" (id 9) (at 346.71 175.26 0)
+      (effects (font (size 1.27 1.27)) hide)
+    )
+    (property "Price@1000pcs" "0,084" (id 10) (at 346.71 175.26 0)
+      (effects (font (size 1.27 1.27)) hide)
+    )
+    (property "Developer" "MW" (id 11) (at 346.71 175.26 0)
+      (effects (font (size 1.27 1.27)) hide)
+    )
+    (property "Package" "0402" (id 12) (at 346.71 175.26 0)
+      (effects (font (size 1.27 1.27)) hide)
+    )
+    (property "LCSC Part #(optional)" "C76890" (id 13) (at 346.71 175.26 0)
+      (effects (font (size 1.27 1.27)) hide)
     )
     (pin "1")
@@
     (pin "1")
   )
-  (symbol (lib_id "Fpc_Connectors:24pin_505110-2491_0.5mm") (at 373.38 119.38 0) (unit 1)
-    (in_bom yes) (on_board yes)
-    (property "Reference" "CON2" (id 0) (at 380.4412 118.0846 0)
-      (effects (font (size 1.27 1.27)) (justify left))
-    )
-    (property "Value" "505110-2491" (id 1) (at 380.4412 120.396 0)
-      (effects (font (size 1.27 1.27)) (justify left))
-    )
-    (property "Footprint" "Fpc_Connectors:505110-2491" (id 2) (at 373.38 110.49 0)
-      (effects (font (size 1.27 1.27)) hide)
-    )
-    (property "Datasheet" "https://pl.mouser.com/datasheet/2/276/2/5051102491_FFC_FPC_CONNECTORS-705759.pdf" (id 3) (at 373.38 110.49 0)
-      (effects (font (size 1.27 1.27)) hide)
-    )
-    (property "Manufacturer" "MOLEX" (id 4) (at 373.38 119.38 0)
-      (effects (font (size 1.27 1.27)) hide)
-    )
-    (property "Manufacturer Part Number" "505110-2491" (id 5) (at 373.38 119.38 0)
-      (effects (font (size 1.27 1.27)) hide)
-    )
-    (property "Supplier" "Mouser" (id 6) (at 373.38 119.38 0)
-      (effects (font (size 1.27 1.27)) hide)
-    )
-    (property "Supplier Part Number" "538-505110-2491" (id 7) (at 373.38 119.38 0)
-      (effects (font (size 1.27 1.27)) hide)
-    )
-    (property "URL" "https://pl.mouser.com/ProductDetail/Molex/505110-2491?qs=fSIr1QPo%2F%2FQZaS1NuXTizw%3D%3D" (id 8) (at 373.38 119.38 0)
-      (effects (font (size 1.27 1.27)) hide)
-    )
-    (property "Price@1pc" "3,13" (id 9) (at 373.38 119.38 0)
-      (effects (font (size 1.27 1.27)) hide)
-    )
-    (property "Price@1000pcs" "1,74" (id 10) (at 373.38 119.38 0)
-      (effects (font (size 1.27 1.27)) hide)
-    )
-    (property "Developer" "MW" (id 11) (at 373.38 119.38 0)
-      (effects (font (size 1.27 1.27)) hide)
-    )
-    (property "Package" "SMD/SMT FPC/FFC" (id 12) (at 373.38 119.38 0)
-      (effects (font (size 1.27 1.27)) hide)
-    )
+  (symbol (lib_id "Fpc_Connectors:24pin_505110-2491_0.5mm") (at 373.38 120.015 0) (unit 1)
+    (in_bom yes) (on_board yes)
+    (property "Reference" "CON2" (id 0) (at 380.4412 118.7196 0)
+      (effects (font (size 1.27 1.27)) (justify left))
+    )
+    (property "Value" "505110-2491" (id 1) (at 380.4412 121.031 0)
+      (effects (font (size 1.27 1.27)) (justify left))
+    )
+    (property "Footprint" "Fpc_Connectors:505110-2491" (id 2) (at 373.38 111.125 0)
+      (effects (font (size 1.27 1.27)) hide)
+    )
+    (property "Datasheet" "https://pl.mouser.com/datasheet/2/276/2/5051102491_FFC_FPC_CONNECTORS-705759.pdf" (id 3) (at 373.38 111.125 0)
+      (effects (font (size 1.27 1.27)) hide)
+    )
+    (property "Manufacturer" "MOLEX" (id 4) (at 373.38 120.015 0)
+      (effects (font (size 1.27 1.27)) hide)
+    )
+    (property "Manufacturer Part Number" "505110-2491" (id 5) (at 373.38 120.015 0)
+      (effects (font (size 1.27 1.27)) hide)
+    )
+    (property "Supplier" "Mouser" (id 6) (at 373.38 120.015 0)
+      (effects (font (size 1.27 1.27)) hide)
+    )
+    (property "Supplier Part Number" "538-505110-2491" (id 7) (at 373.38 120.015 0)
+      (effects (font (size 1.27 1.27)) hide)
+    )
+    (property "URL" "https://pl.mouser.com/ProductDetail/Molex/505110-2491?qs=fSIr1QPo%2F%2FQZaS1NuXTizw%3D%3D" (id 8) (at 373.38 120.015 0)
+      (effects (font (size 1.27 1.27)) hide)
+    )
+    (property "Price@1pc" "3,13" (id 9) (at 373.38 120.015 0)
+      (effects (font (size 1.27 1.27)) hide)
+    )
+    (property "Price@1000pcs" "1,74" (id 10) (at 373.38 120.015 0)
+      (effects (font (size 1.27 1.27)) hide)
+    )
+    (property "Developer" "MW" (id 11) (at 373.38 120.015 0)
+      (effects (font (size 1.27 1.27)) hide)
+    )
+    (property "Package" "SMD/SMT FPC/FFC" (id 12) (at 373.38 120.015 0)
+      (effects (font (size 1.27 1.27)) hide)
+    )
+    (pin "0")
     (pin "1")
     (pin "10")
@@
       (effects (font (size 1.27 1.27)) hide)
     )
+    (pin "0")
     (pin "1")
     (pin "2")
@@
     )
     (pin "1")
+  )
+  (symbol (lib_id "power:GND") (at 284.48 175.26 0) (mirror x) (unit 1)
+    (in_bom yes) (on_board yes)
+    (property "Reference" "#PWR0230" (id 0) (at 284.48 177.8 0)
+      (effects (font (size 0.762 0.762)) hide)
+    )
+    (property "Value" "GND" (id 1) (at 284.48 172.72 0)
+      (effects (font (size 0.762 0.762)) hide)
+    )
+    (property "Footprint" "" (id 2) (at 284.48 175.26 0)
+      (effects (font (size 1.524 1.524)))
+    )
+    (property "Datasheet" "" (id 3) (at 284.48 175.26 0)
+      (effects (font (size 1.524 1.524)))
+    )
+    (pin "1")
+  )
+  (symbol (lib_id "power:GND") (at 364.49 151.13 90) (mirror x) (unit 1)
+    (in_bom yes) (on_board yes)
+    (property "Reference" "#PWR0231" (id 0) (at 361.95 151.13 0)
+      (effects (font (size 0.762 0.762)) hide)
+    )
+    (property "Value" "GND" (id 1) (at 367.03 151.13 0)
+      (effects (font (size 0.762 0.762)) hide)
+    )
+    (property "Footprint" "" (id 2) (at 364.49 151.13 0)
+      (effects (font (size 1.524 1.524)))
+    )
+    (property "Datasheet" "" (id 3) (at 364.49 151.13 0)
+      (effects (font (size 1.524 1.524)))
+    )
+    (pin "1")

Commit message: Eliminated all warnings realted with footprints
Parts:
- C5, C6: footprint Capacitors_Smd_0603:100nF_0603 -> Capacitors_Smd_0402:100nF_0402; symbol Capacitors_Smd0603:100n -> Capacitors_Smd0402:100nF; Developer (none) -> MW; LCSC Part # (optional) (none) -> C131394; Manufacturer SAMSUNG -> Murata; Manufacturer Part Number CL10B104JB8NNNC -> GRM155R71H104KE14D; Package 0603 -> 0402; Package_1 (none) -> 0402; Price@1000pcs 0,02231 -> 0,03299; Price@1pc 0,04540 -> 0,07091; Supplier TME -> Tme; Supplier Part Number CL10B104JB8NNNC -> GRM155R71H104KE14D; URL https://www.tme.eu/pl/details/cl10b104jb8nnnc/kondensatory-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 -> https://www.tme.eu/pl/details/grm155r71h104ke14d/kondensato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
Changed lines of the file:
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@@
     (pin "2")
   )
-  (symbol (lib_id "Capacitors_Smd0603:100n") (at 339.09 213.36 0) (unit 1)
+  (symbol (lib_id "Capacitors_Smd0402:100nF") (at 339.09 213.36 0) (unit 1)
     (in_bom yes) (on_board yes)
     (property "Reference" "C5" (id 0) (at 342.4174 212.1916 0)
@@
       (effects (font (size 1.27 1.27)) (justify left))
     )
-    (property "Footprint" "Capacitors_Smd_0603:100nF_0603" (id 2) (at 339.09 213.36 0)
-      (effects (font (size 1.524 1.524)) hide)
-    )
-    (property "Datasheet" "Capacitors/Smd_0603/Components_Documentation/KEM_C1005_Y5V_SMD.pdf" (id 3) (at 339.09 213.36 0)
-      (effects (font (size 1.524 1.524)) hide)
-    )
-    (property "Manufacturer" "SAMSUNG" (id 4) (at 339.09 213.36 0)
+    (property "Footprint" "Capacitors_Smd_0402:100nF_0402" (id 2) (at 339.09 213.36 0)
       (effects (font (size 1.27 1.27)) hide)
     )
-    (property "Manufacturer Part Number" "CL10B104JB8NNNC" (id 5) (at 339.09 213.36 0)
+    (property "Datasheet" "https://www.tme.eu/Document/558f361ed82994aff5a3e7789d970dd1/GRM155R71H104KE14-01.pdf" (id 3) (at 339.09 213.36 0)
       (effects (font (size 1.27 1.27)) hide)
     )
-    (property "Supplier" "TME" (id 6) (at 339.09 213.36 0)
+    (property "Manufacturer" "Murata" (id 4) (at 339.09 213.36 0)
       (effects (font (size 1.27 1.27)) hide)
     )
-    (property "Supplier Part Number" "CL10B104JB8NNNC" (id 7) (at 339.09 213.36 0)
+    (property "Manufacturer Part Number" "GRM155R71H104KE14D" (id 5) (at 339.09 213.36 0)
       (effects (font (size 1.27 1.27)) hide)
     )
-    (property "URL" "https://www.tme.eu/pl/details/cl10b104jb8nnnc/kondensatory-mlcc-smd-0603/samsung/" (id 8) (at 339.09 213.36 0)
+    (property "Supplier" "Tme" (id 6) (at 339.09 213.36 0)
       (effects (font (size 1.27 1.27)) hide)
     )
-    (property "Price@1pc" "0,04540" (id 9) (at 339.09 213.36 0)
+    (property "Supplier Part Number" "GRM155R71H104KE14D" (id 7) (at 339.09 213.36 0)
       (effects (font (size 1.27 1.27)) hide)
     )
-    (property "Price@1000pcs" "0,02231" (id 10) (at 339.09 213.36 0)
+    (property "URL" "https://www.tme.eu/pl/details/grm155r71h104ke14d/kondensatory-mlcc-smd-0402/murata/" (id 8) (at 339.09 213.36 0)
       (effects (font (size 1.27 1.27)) hide)
     )
-    (property "Package" "0603" (id 11) (at 339.09 213.36 0)
+    (property "Price@1pc" "0,07091" (id 9) (at 339.09 213.36 0)
+      (effects (font (size 1.27 1.27)) hide)
+    )
+    (property "Price@1000pcs" "0,03299" (id 10) (at 339.09 213.36 0)
+      (effects (font (size 1.27 1.27)) hide)
+    )
+    (property "Package" "0402" (id 11) (at 339.09 213.36 0)
+      (effects (font (size 1.27 1.27)) hide)
+    )
+    (property "Developer" "MW" (id 12) (at 339.09 213.36 0)
+      (effects (font (size 1.27 1.27)) hide)
+    )
+    (property "Package_1" "0402" (id 13) (at 339.09 213.36 0)
+      (effects (font (size 1.27 1.27)) hide)
+    )
+    (property "LCSC Part # (optional)" "C131394" (id 14) (at 339.09 213.36 0)
       (effects (font (size 1.27 1.27)) hide)
     )
@@
     (pin "2")
   )
-  (symbol (lib_id "Capacitors_Smd0603:100n") (at 354.33 185.42 0) (unit 1)
+  (symbol (lib_id "Capacitors_Smd0402:100nF") (at 354.33 185.42 0) (unit 1)
     (in_bom yes) (on_board yes)
     (property "Reference" "C6" (id 0) (at 349.25 182.88 0)
@@
       (effects (font (size 1.27 1.27)) (justify left))
     )
-    (property "Footprint" "Capacitors_Smd_0603:100nF_0603" (id 2) (at 354.33 185.42 0)
-      (effects (font (size 1.524 1.524)) hide)
-    )
-    (property "Datasheet" "Capacitors/Smd_0603/Components_Documentation/KEM_C1005_Y5V_SMD.pdf" (id 3) (at 354.33 185.42 0)
-      (effects (font (size 1.524 1.524)) hide)
-    )
-    (property "Manufacturer" "SAMSUNG" (id 4) (at 354.33 185.42 0)
+    (property "Footprint" "Capacitors_Smd_0402:100nF_0402" (id 2) (at 354.33 185.42 0)
       (effects (font (size 1.27 1.27)) hide)
     )
-    (property "Manufacturer Part Number" "CL10B104JB8NNNC" (id 5) (at 354.33 185.42 0)
+    (property "Datasheet" "https://www.tme.eu/Document/558f361ed82994aff5a3e7789d970dd1/GRM155R71H104KE14-01.pdf" (id 3) (at 354.33 185.42 0)
       (effects (font (size 1.27 1.27)) hide)
     )
-    (property "Supplier" "TME" (id 6) (at 354.33 185.42 0)
+    (property "Manufacturer" "Murata" (id 4) (at 354.33 185.42 0)
       (effects (font (size 1.27 1.27)) hide)
     )
-    (property "Supplier Part Number" "CL10B104JB8NNNC" (id 7) (at 354.33 185.42 0)
+    (property "Manufacturer Part Number" "GRM155R71H104KE14D" (id 5) (at 354.33 185.42 0)
       (effects (font (size 1.27 1.27)) hide)
     )
-    (property "URL" "https://www.tme.eu/pl/details/cl10b104jb8nnnc/kondensatory-mlcc-smd-0603/samsung/" (id 8) (at 354.33 185.42 0)
+    (property "Supplier" "Tme" (id 6) (at 354.33 185.42 0)
       (effects (font (size 1.27 1.27)) hide)
     )
-    (property "Price@1pc" "0,04540" (id 9) (at 354.33 185.42 0)
+    (property "Supplier Part Number" "GRM155R71H104KE14D" (id 7) (at 354.33 185.42 0)
       (effects (font (size 1.27 1.27)) hide)
     )
-    (property "Price@1000pcs" "0,02231" (id 10) (at 354.33 185.42 0)
+    (property "URL" "https://www.tme.eu/pl/details/grm155r71h104ke14d/kondensatory-mlcc-smd-0402/murata/" (id 8) (at 354.33 185.42 0)
       (effects (font (size 1.27 1.27)) hide)
     )
-    (property "Package" "0603" (id 11) (at 354.33 185.42 0)
+    (property "Price@1pc" "0,07091" (id 9) (at 354.33 185.42 0)
       (effects (font (size 1.27 1.27)) hide)
     )
+    (property "Price@1000pcs" "0,03299" (id 10) (at 354.33 185.42 0)
+      (effects (font (size 1.27 1.27)) hide)
+    )
+    (property "Package" "0402" (id 11) (at 354.33 185.42 0)
+      (effects (font (size 1.27 1.27)) hide)
+    )
+    (property "Developer" "MW" (id 12) (at 354.33 185.42 0)
+      (effects (font (size 1.27 1.27)) hide)
+    )
+    (property "Package_1" "0402" (id 13) (at 354.33 185.42 0)
+      (effects (font (size 1.27 1.27)) hide)
+    )
+    (property "LCSC Part # (optional)" "C131394" (id 14) (at 354.33 185.42 0)
+      (effects (font (size 1.27 1.27)) hide)
+    )
