File: ethernet.kicad_sch (KiCad schematic)
At the start: 42 parts, among them T2 WE-RJ45_74990101210, U7 KSZ8041NL_RNL, X2 ECS-2016MV-250-CN-TR

Commit message: Reworked schematic and applied changes on pcb related with mini pci express
Parts:
- C33, C38: symbol Capacitors_Smd_Tantal:22uF6V3 -> Capacitors_Smd_Tantal:22uF_10V; Developer (none) -> MW; LCSC Part #(optional) (none) -> C123266; Manufacturer (none) -> VISHAY; Manufacturer Part Number (none) -> 293D226X9010C2TE3; Package (none) -> 2312/Size_C; Price@1000pcs (none) -> 0,43; Price@1pc (none) -> 0,9; Supplier (none) -> TME; Supplier Part Number (none) -> 293D226X9010C2TE3; URL (none) -> https://www.tme.eu/pl/en/details/293d226x9010c2te3/smd-tant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
- C34, C35, C36, C37, C40, C41, C42, C43: symbol Capacitors_Smd0402:100nF -> Capacitors_Smd0603:100n; Manufacturer Murata -> SAMSUNG; Manufacturer Part Number GRM155R71H104KE14D -> CL10B104JB8NNNC; Package 0402 -> 0603; Price@1000pcs 0,03299 -> 0,02231; Price@1pc 0,07091 -> 0,04540; Supplier Tme -> TME; Supplier Part Number GRM155R71H104KE14D -> CL10B104JB8NNNC; URL https://www.tme.eu/pl/details/grm155r71h104ke14d/kondensato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 -> https://www.tme.eu/pl/details/cl10b104jb8nnnc/kondensatory-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
Connections:
- no-connect marks 6 -> 5

Commit message: Modified ethernet
Parts:
- removed R37, R39: 1k, Resistor_Smd_0603:1k_0603, symbol Resistors_Smd0603:1k_0603
- removed R38: 4k7_NM, Resistor_Smd_0603:4k7_0603, symbol Resistors_Smd0603:4k7
- added R?: 4k7_NM, Resistor_Smd_0603:4k7_0603, symbol Resistors_Smd0603:4k7
- added R? (x2): 1k, Resistor_Smd_0603:1k_0603, symbol Resistors_Smd0603:1k_0603
Connections:
- net 3V3: now also R?.1
- net GND: now also R?.2, R?.2
- net ENET-COL: now reaches U7.28 (COL/CONFIG0)
- net ENET-COL: now also R?.1, R?.2
- net ENET-CRS: now reaches U7.29 (CRS/CONFIG1)
- net ENET-CRS: now also R?.1
- net ENET-RX-CLK: now reaches U7.19 (RXC)
- net ENET-TX-CLK: now reaches U7.22 (TXC)
- net ENET-REFCLK: no longer names the net of R41.1, U7.9 (XI_/REFCLK)
- net ENET_MDC renamed ENET-MDC
- no-connect marks 5 -> 3
Other:
- moved on the sheet: R27, R42, R43, R44, R45, R46, R47

Commit message: Started etherner reworking
Parts:
- gave numbers to parts that had none: 3
Changed lines of the file:
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@@
   (symbol (lib_id "power:GND") (at 260.35 91.44 270) (unit 1)
     (in_bom yes) (on_board yes)
-    (property "Reference" "#PWR?" (id 0) (at 262.89 91.44 0)
+    (property "Reference" "#PWR0198" (id 0) (at 262.89 91.44 0)
       (effects (font (size 0.762 0.762)) hide)
     )
@@
   (symbol (lib_id "power:GND") (at 260.35 105.41 270) (unit 1)
     (in_bom yes) (on_board yes)
-    (property "Reference" "#PWR?" (id 0) (at 262.89 105.41 0)
+    (property "Reference" "#PWR0177" (id 0) (at 262.89 105.41 0)
       (effects (font (size 0.762 0.762)) hide)
     )
@@
   (symbol (lib_id "power:3V3_NO_GLOBAL") (at 259.08 101.6 270) (unit 1)
     (in_bom yes) (on_board yes)
-    (property "Reference" "#PWR?" (id 0) (at 261.62 101.6 0)
+    (property "Reference" "#PWR71" (id 0) (at 261.62 101.6 0)
       (effects (font (size 1.016 1.016)) hide)
     )
@@
   (symbol (lib_id "Resistors_Smd0603:1k_0603") (at 251.46 91.44 90) (unit 1)
     (in_bom yes) (on_board yes)
-    (property "Reference" "R?" (id 0) (at 252.73 88.9 90)
+    (property "Reference" "R37" (id 0) (at 252.73 88.9 90)
       (effects (font (size 1.27 1.27)) (justify left))
     )
@@
   (symbol (lib_id "Resistors_Smd0603:4k7") (at 251.46 101.6 270) (unit 1)
     (in_bom yes) (on_board yes)
-    (property "Reference" "R?" (id 0) (at 257.81 100.33 90))
+    (property "Reference" "R38" (id 0) (at 257.81 100.33 90))
     (property "Value" "4k7_NM" (id 1) (at 251.46 101.6 90))
     (property "Footprint" "Resistor_Smd_0603:4k7_0603" (id 2) (at 251.46 101.6 0)
@@
   (symbol (lib_id "Resistors_Smd0603:1k_0603") (at 251.46 105.41 90) (unit 1)
     (in_bom yes) (on_board yes)
-    (property "Reference" "R?" (id 0) (at 259.08 104.14 90)
-      (effects (font (size 1.27 1.27)) (justify left))
-    )
+    (property "Reference" "R39" (id 0) (at 259.08 104.14 90)
+      (effects (font (size 1.27 1.27)) (justify left))
+    )

Commit message: Added some rules for ethernet
Other:
- note added: "MII and RMII Routing Guidelines All connections on a PCB in MII and RMII routing are point-to-point connections. Although MII and RMII use relatively low data rates, the limiting parameter that determines whether a trace can act as a transmission line is the signal rise/fall time. Unless your board is very large or your signal switching speed is very fast, reflections at the end of each connectio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"
- note added: "Track width 4.75mil for all"
Changed lines of the file:
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@@
     )
+  )
+  (text "MII and RMII Routing Guidelines\n\nAll connections on a PCB in MII and RMII routing are point-to-point connections. Although MII and RMII use relatively low data rates, \nthe limiting parameter that determines whether a trace can act as a transmission line is the signal rise/fall time. Unless your board \nis very large or your signal switching speed is very fast, reflections at the end of each connection can be ignored. \nThe recommended trace impedance in MII is 50 Ohms +/- 10%.\nAlthough the trace length between the PHY and MAC is generally short enough to ignore transmission line effects,\nyou should pay attention to impedance when routing the signal and clock traces when the traces are electrically long. \nSince MII and RMII require clock signals between the PHY and MAC, best practices for routing clock signals should be used \nwith longer traces. Generally, you should avoid the use of vias on traces carrying clock signals on board with impedance control \nas the trace impedance can be different between layers. However, as long as the impedance in each layer is carefully controlled to the\nright value, then the clock signals can certainly be routed through vias. This will prevent signal reflections on longer clock traces.\nFor the above reasons, all MII/RMII signal traces should be routed as short as possible on a single layer, and traces should be\nrouted in a straight path. If you must turn a corner with a signal trace, the trace should bend by no more than 45 degrees.\nClock lines should also be shielded with GND lines to prevent crosstalk through capacitive coupling,\nespecially when longer traces are necessary. Because the TX and RX data signals are triggered by the rising edge of the clock,\ncommunication in MII and RMII is synchronous. Thus, the data lines and the clock line between the MAC and PHY should be length matched.\nThe allowed deviation in length matching depends on the rise/fall time for digital signals between these two elements, \nalthough it is generally recommended that any deviation be less than 10 mm as MII and RMII use TTL logic.\nAgain, the allowed trace length mismatch depends on the rise/fall time of digital signals."
+    (at 17.78 278.13 0)
+    (effects (font (size 1.27 1.27)) (justify left bottom))
+  )
+  (text "Track width 4.75mil for all" (at 44.45 226.06 180)
+    (effects (font (size 1.27 1.27)) (justify right bottom))
   )
   (label "ETH_RX_N" (at 318.77 124.46 0)

Commit message: Updated schematic
Changed lines of the file:
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@@
-(kicad_sch (version 20210406) (generator eeschema)
+(kicad_sch (version 20210615) (generator eeschema)
   (paper "A3")
   (title_block
