File: ethernet.kicad_sch (KiCad schematic)
At the start: 42 parts, among them T2 WE-RJ45_74990101210, U7 KSZ8041NL_RNL, X2 ECS-2016MV-250-CN-TR

Commit message: Corrected schematic
Parts:
- removed C36: 100nF/50V, Capacitors_Smd_0402:100nF_0402, symbol Capacitors_Smd0603:100n
- removed C39: 1uF/10V, Capacitors_Smd_0402:1uF_0402, symbol Capacitors_Smd0402:1uF
- removed R25, R27, R28, R34, R35: 1k, Resistor_Smd_0603:1k_0603, symbol Resistors_Smd0603:1k_0603
- removed X2: ECS-2016MV-250-CN-TR, Resonators:520-2016MV-250-CNT, symbol Resonators:ECS-2016MV-250-CN-TR
- added R25, R27, R28, R35: 4k7, Resistor_Smd_0603:4k7_0603, symbol Resistors_Smd0603:4k7
- added R34, R64, R67, R70: 33R, Resistor_Smd_0402:33R_0402, symbol Resistors_Smd0402:33R
- added R71, R72: 10R, Resistor_Smd_0402:10R_0402, symbol Resistors_Smd0402:10R
Connections:
- net 3V3: now also C38.1, U7.17 (VDDIO_3.3), R25.1, R27.1, R28.1, R35.1; no longer U7.3 (VDDA_3.3)
- net ENET-IRQ: now also R27.2
- net ENET-MDIO: now also R35.2
- net ENET-RXD0: now also R70.2; no longer U7.16 (RXD0/RXD[0]/DUPLEX)
- net ENET-RXD1: now also R67.2; no longer U7.15 (RXD1/RXD[1]/PHYAD2)
- net ENET-TXD0: now also R64.2; no longer U7.24 (TXD0/TXD[0])
- net ENET-TXD1: now also R34.2; no longer U7.25 (TXD1/TXD[1])
- net ENET-~{RST}: now reaches R40.2, U7.32 (~{RST})
- net at C37.1, L7.2: now also U7.3 (VDDA_3.3), R71.1, R72.1; no longer C38.1, U7.17 (VDDIO_3.3)
- net ENET-CLK: now reaches R41.2
- net at C43.2, T2.5 (CRD): now also R71.2
- net at C42.2, T2.4 (CTD): now also R72.2
- net ENET-COL: no longer names the net of R38.2, R39.1, U7.28 (COL/CONFIG0)
- net ENET-CRS: no longer names the net of R37.1, U7.29 (CRS/CONFIG1)
- net ENET-RX-CLK: no longer names the net of U7.19 (RXC)
- net ENET-RXD2: no longer names the net of R29.2, U7.14 (RXD2/PHYAD1)
- net ENET-RXD3: no longer names the net of U7.13 (RXD3_/PHYAD0)
- net ENET-RXD3: now also R28.2
- net ENET-RXER: no longer names the net of R30.2
- net ENET-RXER: now also R25.2
- net ENET-TX-CLK: no longer names the net of U7.22 (TXC)
- net ENET-TXD2: no longer names the net of U7.26 (TXD2)
- net ENET-TXD3: no longer names the net of U7.27 (TXD3)
- new net: R67.1, U7.15 (RXD1/RXD[1]/PHYAD2)
- new net: R70.1, U7.16 (RXD0/RXD[0]/DUPLEX)
- new net: R64.1, U7.24 (TXD0/TXD[0])
- new net: R34.1, U7.25 (TXD1/TXD[1])
- no-connect marks 3 -> 7
Other:
- moved on the sheet: C37, C38, C42, C43, R40, R41

Commit message: Cleared all errors DRC
Parts:
- C34, C35, C37, C40, C41, C42, C43: footprint Capacitors_Smd_0402:100nF_0402 -> Capacitors_Smd_0603:100nF_0603
- R40: Developer (none) -> MW; LCSC Part #(optional) (none) -> C269684; Manufacturer (none) -> ROYAL OHM; Manufacturer Part Number (none) -> 0603SAJ0103T5E; Package (none) -> 0603; Price@1000pcs (none) -> 0,01111; Price@1pc (none) -> 0,04560; Supplier (none) -> TME; Supplier Part Number (none) -> SMD0603-10K; URL (none) -> https://www.tme.eu/pl/details/smd0603-10k/rezystory-smd-060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
Changed lines of the file:
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@@
       (effects (font (size 1.524 1.524)) (justify left) hide)
+    )
+    (property "Manufacturer" "ROYAL OHM" (id 4) (at 248.92 161.925 0)
+      (effects (font (size 1.27 1.27)) hide)
+    )
+    (property "Manufacturer Part Number" "0603SAJ0103T5E" (id 5) (at 248.92 161.925 0)
+      (effects (font (size 1.27 1.27)) hide)
+    )
+    (property "Supplier" "TME" (id 6) (at 248.92 161.925 0)
+      (effects (font (size 1.27 1.27)) hide)
+    )
+    (property "Supplier Part Number" "SMD0603-10K" (id 7) (at 248.92 161.925 0)
+      (effects (font (size 1.27 1.27)) hide)
+    )
+    (property "URL" "https://www.tme.eu/pl/details/smd0603-10k/rezystory-smd-0603/royal-ohm/0603saj0103t5e/" (id 8) (at 248.92 161.925 0)
+      (effects (font (size 1.27 1.27)) hide)
+    )
+    (property "Price@1pc" "0,04560" (id 9) (at 248.92 161.925 0)
+      (effects (font (size 1.27 1.27)) hide)
+    )
+    (property "Price@1000pcs" "0,01111" (id 10) (at 248.92 161.925 0)
+      (effects (font (size 1.27 1.27)) hide)
+    )
+    (property "Developer" "MW" (id 11) (at 248.92 161.925 0)
+      (effects (font (size 1.27 1.27)) hide)
+    )
+    (property "Package" "0603" (id 12) (at 248.92 161.925 0)
+      (effects (font (size 1.27 1.27)) hide)
+    )
+    (property "LCSC Part #(optional)" "C269684" (id 13) (at 248.92 161.925 0)
+      (effects (font (size 1.27 1.27)) hide)
     )
     (pin "1")
@@
       (effects (font (size 1.27 1.27)) (justify left))
     )
-    (property "Footprint" "Capacitors_Smd_0402:100nF_0402" (id 2) (at 364.49 50.8 0)
+    (property "Footprint" "Capacitors_Smd_0603:100nF_0603" (id 2) (at 364.49 50.8 0)
       (effects (font (size 1.524 1.524)) hide)
     )
@@
       (effects (font (size 1.27 1.27)) (justify left))
     )
-    (property "Footprint" "Capacitors_Smd_0402:100nF_0402" (id 2) (at 190.5 50.8 0)
+    (property "Footprint" "Capacitors_Smd_0603:100nF_0603" (id 2) (at 190.5 50.8 0)
       (effects (font (size 1.524 1.524)) hide)
     )
@@
       (effects (font (size 1.27 1.27)) (justify left))
     )
-    (property "Footprint" "Capacitors_Smd_0402:100nF_0402" (id 2) (at 153.67 69.85 0)
+    (property "Footprint" "Capacitors_Smd_0603:100nF_0603" (id 2) (at 153.67 69.85 0)
       (effects (font (size 1.524 1.524)) hide)
     )
@@
       (effects (font (size 1.27 1.27)) (justify left))
     )
-    (property "Footprint" "Capacitors_Smd_0402:100nF_0402" (id 2) (at 302.26 176.53 0)
+    (property "Footprint" "Capacitors_Smd_0603:100nF_0603" (id 2) (at 302.26 176.53 0)
       (effects (font (size 1.524 1.524)) hide)
     )
@@
       (effects (font (size 1.27 1.27)) (justify left))
     )
-    (property "Footprint" "Capacitors_Smd_0402:100nF_0402" (id 2) (at 284.48 176.53 0)
+    (property "Footprint" "Capacitors_Smd_0603:100nF_0603" (id 2) (at 284.48 176.53 0)
       (effects (font (size 1.524 1.524)) hide)
     )
@@
       (effects (font (size 1.27 1.27)) (justify left))
     )
-    (property "Footprint" "Capacitors_Smd_0402:100nF_0402" (id 2) (at 334.01 129.54 0)
+    (property "Footprint" "Capacitors_Smd_0603:100nF_0603" (id 2) (at 334.01 129.54 0)
       (effects (font (size 1.524 1.524)) hide)
     )
@@
       (effects (font (size 1.27 1.27)) (justify left))
     )
-    (property "Footprint" "Capacitors_Smd_0402:100nF_0402" (id 2) (at 334.01 139.7 0)
-      (effects (font (size 1.524 1.524)) hide)
-    )
+    (property "Footprint" "Capacitors_Smd_0603:100nF_0603" (id 2) (at 334.01 139.7 0)
+      (effects (font (size 1.524 1.524)) hide)
+    )

Commit message: Eliminated all warnings realted with footprints
Parts:
- C34, C35, C37, C40, C41, C42, C43: footprint Capacitors_Smd_0603:100nF_0603 -> Capacitors_Smd_0402:100nF_0402; symbol Capacitors_Smd0603:100n -> Capacitors_Smd0402:100nF; Manufacturer SAMSUNG -> Murata; Manufacturer Part Number CL10B104JB8NNNC -> GRM155R71H104KE14D; Package 0603 -> 0402; Package_1 (none) -> 0402; Price@1000pcs 0,02231 -> 0,03299; Price@1pc 0,04540 -> 0,07091; Supplier TME -> Tme; Supplier Part Number CL10B104JB8NNNC -> GRM155R71H104KE14D; URL https://www.tme.eu/pl/details/cl10b104jb8nnnc/kondensatory-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 -> https://www.tme.eu/pl/details/grm155r71h104ke14d/kondensato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

Commit message: Gerbers created, BOM, CPL
Parts:
- L7: Developer (none) -> MW; LCSC Part #(optional) (none) -> C14709; Manufacturer (none) -> MURATA; Manufacturer Part Number (none) -> BLM18PG121SN1D; Package (none) -> 0603; Price@1000pcs (none) -> 0,08394; Price@1pc (none) -> 0,20599; Supplier (none) -> Tme; Supplier Part Number (none) -> BLM18PG121SN1D; URL (none) -> https://www.tme.eu/pl/details/blm18pg121sn1d/ferryty-korali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
- R25, R27, R28, R35, R38, R42, R43: Manufacturer (none) -> ROYAL OHM; Manufacturer Part Number (none) -> 0603SAF4701T5E; Package (none) -> 0603; Price@1000pcs (none) -> 0,01271; Price@1pc (none) -> 0,04698; Supplier (none) -> TME; Supplier Part Number (none) -> SMD0603-4K7-1%; URL (none) -> https://www.tme.eu/pl/details/smd0603-4k7-1%2525/rezystory-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
- R26, R29, R31, R32, R37, R39, R44, R45: Manufacturer (none) -> ROYAL OHM; Manufacturer Part Number (none) -> 0603SAF1001T5E; Package (none) -> 0603; Price@1000pcs (none) -> 0,01269; Price@1pc (none) -> 0,04693; Supplier (none) -> TME; Supplier Part Number (none) -> SMD0603-1K-1%; URL (none) -> https://www.tme.eu/pl/details/smd0603-1k-1%2525/rezystory-s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
- R36: symbol Resistors_Smd0603:6k49_0603 -> Resistors_Smd0603:6k49; Developer (none) -> MW; LCSC Part #(optional) (none) -> C269508; Manufacturer (none) -> ROYAL OHM; Manufacturer Part Number (none) -> 0603SAF6491T5E; Package (none) -> 0603; Price@1000pcs (none) -> 0.01330; Price@1pc (none) -> 0.04826; Supplier (none) -> Tme; Supplier Part Number (none) -> SMD0603-6K49-1%; URL (none) -> https://www.tme.eu/pl/details/smd0603-6k49-1%25/rezystory-s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

Commit message: Changed ethernet connector to horizontal and changed it position to avoid collision with arduino shield
Parts:
- removed T2: WE-RJ45_74990101210, RJ45_Ethernet_Transformer:WE-RJ45_74990101210, symbol RJ45_Ethernet_Transformer:WE-RJ45_74990101210
- added CON7: LMJ3628844TA753, RJ45_Ethernet_Transformer:LMJ3628844TA753, symbol RJ45_Ethernet_Transformer:LMJ3628844TA753
Connections:
- net 3V3: now also CON7.12, CON7.9
- net ETH_RX_N: now also CON7.P6
- net ETH_RX_P: now also CON7.P3
- net ETH_TX_N: now also CON7.P2
- net ETH_TX_P: now also CON7.P1
- net GND: now also CON7.0, CON7.P8
- net at R47.1: now also CON7.10
- net at R46.1: now also CON7.11
- net at C43.2, R71.2: now also CON7.P5
- net at C42.2, R72.2: now also CON7.P4
- no-connect marks 7 -> 5
Other:
- moved on the sheet: C33, C34, C35, C37, C38, C40, C41, C42, C43, L7, R25, R26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
