File: minipci_module.kicad_sch (KiCad schematic)
At the start: 3 parts, among them Con3 2041119-1

Commit message: Started issues implementation
Parts:
- removed R58, R59: 4k7, Resistor_Smd_0603:4k7_0603, symbol Resistors_Smd0603:4k7
Connections:
- net PCM_IN is gone; now on net SPI_MOSI: Con3.49
- net PCM_OUT is gone; now on net SPI_MISO: Con3.47
- net PCM_SYNC is gone; now on net SPI_GSN: Con3.51
- net TRX_SWITCH-PCM_CLK is gone; now on net SPI_SCK: Con3.45
- net UART_RI is gone; now on net SPDT_SEL-~WDISABLE~: Con3.17
- net GND: no longer Con3.18
- net GPS_PPS: now also Con3.19; no longer Con3.8
- net SPDT_SEL-~WDISABLE~: no longer Con3.20
- net SPI_GSN: no longer Con3.10
- net SPI_MISO: no longer Con3.14
- net SPI_MOSI: no longer Con3.12
- net SPI_SCK: no longer Con3.16
- net I2C-SCL: no longer names the net of Con3.30
- net I2C-SDA: no longer names the net of Con3.32
- net NETLIGHT: no longer names the net of Con3.42
- net PWRKEY: no longer names the net of Con3.1
- net UART_CTS: no longer names the net of Con3.23
- net UART_DCD: no longer names the net of Con3.33
- net UART_DTR: no longer names the net of Con3.31
- net UART_RTS: no longer names the net of Con3.25
- net UART_RX: no longer names the net of Con3.11
- net UART_TX: no longer names the net of Con3.13
- no-connect marks 9 -> 25

Commit message: Tracking finished
Connections:
- net USB-D_M: no longer names the net of Con3.36
- net USB-D_P: no longer names the net of Con3.38
- no-connect marks 25 -> 27
Changed lines of the file:
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@@
   (no_connect (at 189.23 157.48))
   (no_connect (at 189.23 160.02))
+  (no_connect (at 189.23 167.64))
+  (no_connect (at 189.23 172.72))
   (no_connect (at 189.23 182.88))
   (no_connect (at 189.23 187.96))
@@
     (stroke (width 0) (type solid) (color 0 0 0 0))
   )
-  (wire (pts (xy 189.23 167.64) (xy 179.07 167.64))
-    (stroke (width 0) (type solid) (color 0 0 0 0))
-  )
   (wire (pts (xy 189.23 170.18) (xy 186.69 170.18))
-    (stroke (width 0) (type solid) (color 0 0 0 0))
-  )
-  (wire (pts (xy 189.23 172.72) (xy 179.07 172.72))
     (stroke (width 0) (type solid) (color 0 0 0 0))
   )
@@
     (effects (font (size 1.27 1.27)) (justify right))
   )
-  (hierarchical_label "USB-D_M" (shape bidirectional) (at 179.07 167.64 180)
-    (effects (font (size 1.27 1.27)) (justify right))
-  )
-  (hierarchical_label "USB-D_P" (shape bidirectional) (at 179.07 172.72 180)
-    (effects (font (size 1.27 1.27)) (justify right))
-  )

Commit message: Reworked schematic and applied changes on pcb related with mini pci express
Connections:
- net SCL: now reaches Con3.30
- net SDA: now reaches Con3.32
- net GPS_PPS renamed GPS_PPS/UART_TX
- net SPDT_SEL-~WDISABLE~ renamed SPDT_SEL-~WDISABLE~/UART_RX
- no-connect marks 27 -> 25
Changed lines of the file:
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@@
   (no_connect (at 189.23 139.7))
   (no_connect (at 189.23 147.32))
-  (no_connect (at 189.23 152.4))
   (no_connect (at 189.23 154.94))
-  (no_connect (at 189.23 157.48))
   (no_connect (at 189.23 160.02))
   (no_connect (at 189.23 167.64))
@@
   )
   (wire (pts (xy 67.31 40.64) (xy 64.77 40.64))
+    (stroke (width 0) (type solid) (color 0 0 0 0))
+  )
+  (wire (pts (xy 179.07 157.48) (xy 189.23 157.48))
     (stroke (width 0) (type solid) (color 0 0 0 0))
   )
@@
   )
   (wire (pts (xy 189.23 149.86) (xy 186.69 149.86))
+    (stroke (width 0) (type solid) (color 0 0 0 0))
+  )
+  (wire (pts (xy 189.23 152.4) (xy 179.07 152.4))
     (stroke (width 0) (type solid) (color 0 0 0 0))
   )
@@
     (effects (font (size 1.27 1.27)) (justify right))
   )
-  (hierarchical_label "SPDT_SEL-~WDISABLE~" (shape input) (at 179.07 119.38 180)
+  (hierarchical_label "SPDT_SEL-~WDISABLE~{slash}UART_RX" (shape bidirectional) (at 179.07 119.38 180)
     (effects (font (size 1.27 1.27)) (justify right))
   )
-  (hierarchical_label "GPS_PPS" (shape input) (at 179.07 124.46 180)
+  (hierarchical_label "GPS_PPS{slash}UART_TX" (shape bidirectional) (at 179.07 124.46 180)
     (effects (font (size 1.27 1.27)) (justify right))
   )
@@
     (effects (font (size 1.27 1.27)) (justify right))
   )
+  (hierarchical_label "SCL" (shape bidirectional) (at 179.07 152.4 180)
+    (effects (font (size 1.27 1.27)) (justify right))
+  )
+  (hierarchical_label "SDA" (shape bidirectional) (at 179.07 157.48 180)
+    (effects (font (size 1.27 1.27)) (justify right))
+  )

Commit message: Updated schematic
Connections:
- net SPDT_SEL-~WDISABLE~/UART_RX renamed SPDT_SEL-~{WDISABLE}/UART_RX
- net ~RESET~ renamed ~{RESET}
Changed lines of the file:
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@@
-(kicad_sch (version 20210406) (generator eeschema)
+(kicad_sch (version 20210615) (generator eeschema)
   (paper "A3")
   (title_block
@@
     (effects (font (size 1.27 1.27)) (justify right))
   )
-  (hierarchical_label "SPDT_SEL-~WDISABLE~{slash}UART_RX" (shape bidirectional) (at 179.07 119.38 180)
+  (hierarchical_label "SPDT_SEL-~{WDISABLE}{slash}UART_RX" (shape bidirectional) (at 179.07 119.38 180)
     (effects (font (size 1.27 1.27)) (justify right))
   )
@@
     (effects (font (size 1.27 1.27)) (justify right))
   )
-  (hierarchical_label "~RESET~" (shape input) (at 179.07 132.08 180)
+  (hierarchical_label "~{RESET}" (shape input) (at 179.07 132.08 180)
     (effects (font (size 1.27 1.27)) (justify right))
   )
