File: stm32mp1-custom-devboard.kicad_sch (KiCad schematic)
At the start: 20 parts, among them P1 Main Power Supply, Sw1 434153017835, Sw2 434153017835, U10 APX803D-29SRG-7

Commit message: Applied all changes, tunnign started
Parts:
- added R58, R59: 10k, Resistor_Smd_0603:10k_0603, symbol Resistors_Smd0603:10k
Connections:
- net GND: now also R58.1, R59.1
- net STLink Module/STLINK_RX: now also R59.2
- net STLink Module/STLINK_TX: now also R58.2
Changed lines of the file:
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@@
   (junction (at 109.22 43.18) (diameter 1.016) (color 0 0 0 0))
   (junction (at 172.72 76.2) (diameter 1.016) (color 0 0 0 0))
+  (junction (at 261.62 102.87) (diameter 1.016) (color 0 0 0 0))
+  (junction (at 261.62 105.41) (diameter 1.016) (color 0 0 0 0))
   (no_connect (at 158.75 118.11))
   (no_connect (at 158.75 120.65))
@@
     (stroke (width 0) (type solid) (color 0 0 0 0))
   )
+  (wire (pts (xy 246.38 100.33) (xy 243.84 100.33))
+    (stroke (width 0) (type solid) (color 0 0 0 0))
+  )
+  (wire (pts (xy 246.38 107.95) (xy 243.84 107.95))
+    (stroke (width 0) (type solid) (color 0 0 0 0))
+  )
   (wire (pts (xy 252.73 227.33) (xy 254 227.33))
     (stroke (width 0) (type solid) (color 0 0 0 0))
@@
     (stroke (width 0) (type solid) (color 0 0 0 0))
   )
+  (wire (pts (xy 259.08 100.33) (xy 261.62 100.33))
+    (stroke (width 0) (type solid) (color 0 0 0 0))
+  )
+  (wire (pts (xy 259.08 107.95) (xy 261.62 107.95))
+    (stroke (width 0) (type solid) (color 0 0 0 0))
+  )
+  (wire (pts (xy 261.62 100.33) (xy 261.62 102.87))
+    (stroke (width 0) (type solid) (color 0 0 0 0))
+  )
+  (wire (pts (xy 261.62 102.87) (xy 238.76 102.87))
+    (stroke (width 0) (type solid) (color 0 0 0 0))
+  )
+  (wire (pts (xy 261.62 105.41) (xy 238.76 105.41))
+    (stroke (width 0) (type solid) (color 0 0 0 0))
+  )
+  (wire (pts (xy 261.62 107.95) (xy 261.62 105.41))
+    (stroke (width 0) (type solid) (color 0 0 0 0))
+  )
   (wire (pts (xy 264.16 227.33) (xy 265.43 227.33))
     (stroke (width 0) (type solid) (color 0 0 0 0))
@@
     (stroke (width 0) (type solid) (color 0 0 0 0))
   )
-  (wire (pts (xy 270.51 102.87) (xy 238.76 102.87))
+  (wire (pts (xy 270.51 102.87) (xy 261.62 102.87))
     (stroke (width 0) (type solid) (color 0 0 0 0))
   )
-  (wire (pts (xy 270.51 105.41) (xy 238.76 105.41))
+  (wire (pts (xy 270.51 105.41) (xy 261.62 105.41))
     (stroke (width 0) (type solid) (color 0 0 0 0))
   )
@@
     (pin "1")
   )
+  (symbol (lib_id "power:GND") (at 243.84 100.33 270) (unit 1)
+    (in_bom yes) (on_board yes)
+    (property "Reference" "#PWR0200" (id 0) (at 246.38 100.33 0)
+      (effects (font (size 0.762 0.762)) hide)
+    )
+    (property "Value" "GND" (id 1) (at 241.3 100.33 0)
+      (effects (font (size 0.762 0.762)) hide)
+    )
+    (property "Footprint" "" (id 2) (at 243.84 100.33 0)
+      (effects (font (size 1.524 1.524)))
+    )
+    (property "Datasheet" "" (id 3) (at 243.84 100.33 0)
+      (effects (font (size 1.524 1.524)))
+    )
+    (pin "1")
+  )
+  (symbol (lib_id "power:GND") (at 243.84 107.95 270) (unit 1)
+    (in_bom yes) (on_board yes)
+    (property "Reference" "#PWR0208" (id 0) (at 246.38 107.95 0)
+      (effects (font (size 0.762 0.762)) hide)
+    )
+    (property "Value" "GND" (id 1) (at 241.3 107.95 0)
+      (effects (font (size 0.762 0.762)) hide)
+    )
+    (property "Footprint" "" (id 2) (at 243.84 107.95 0)
+      (effects (font (size 1.524 1.524)))
+    )
+    (property "Datasheet" "" (id 3) (at 243.84 107.95 0)
+      (effects (font (size 1.524 1.524)))
+    )
+    (pin "1")
+  )
   (symbol (lib_id "power:GND") (at 267.97 45.72 90) (unit 1)
     (in_bom yes) (on_board yes)
@@
     (pin "2")
   )
+  (symbol (lib_id "Resistors_Smd0603:10k") (at 252.73 100.33 90) (unit 1)
+    (in_bom yes) (on_board yes)
+    (property "Reference" "R58" (id 0) (at 255.3716 97.3328 90)
+      (effects (font (size 1.27 1.27)) (justify left))
+    )
+    (property "Value" "10k" (id 1) (at 254.508 100.5078 90)
+      (effects (font (size 1.27 1.27)) (justify left))
+    )
+    (property "Footprint" "Resistor_Smd_0603:10k_0603" (id 2) (at 252.73 100.33 0)
+      (effects (font (size 1.524 1.524)) hide)
+    )
+    (property "Datasheet" "Resistors/Smd_0603/Components_Documentation/Vishay_Resistors_SM0603.pdf" (id 3) (at 252.73 100.33 0)
+      (effects (font (size 1.524 1.524)) hide)
+    )
+    (property "Manufacturer" "ROYAL OHM" (id 4) (at 252.73 100.33 0)
+      (effects (font (size 1.27 1.27)) hide)
+    )
+    (property "Manufacturer Part Number" "0603SAJ0103T5E" (id 5) (at 252.73 100.33 0)
+      (effects (font (size 1.27 1.27)) hide)
+    )
+    (property "Supplier" "TME" (id 6) (at 252.73 100.33 0)
+      (effects (font (size 1.27 1.27)) hide)
+    )
+    (property "Supplier Part Number" "SMD0603-10K" (id 7) (at 252.73 100.33 0)
+      (effects (font (size 1.27 1.27)) hide)
+    )
+    (property "URL" "https://www.tme.eu/pl/details/smd0603-10k/rezystory-smd-0603/royal-ohm/0603saj0103t5e/" (id 8) (at 252.73 100.33 0)
+      (effects (font (size 1.27 1.27)) hide)
+    )
+    (property "Price@1pc" "0,04560" (id 9) (at 252.73 100.33 0)
+      (effects (font (size 1.27 1.27)) hide)
+    )
+    (property "Price@1000pcs" "0,01111" (id 10) (at 252.73 100.33 0)
+      (effects (font (size 1.27 1.27)) hide)
+    )
+    (property "Developer" "MW" (id 11) (at 252.73 100.33 0)
+      (effects (font (size 1.27 1.27)) hide)
+    )
+    (property "Package" "0603" (id 12) (at 252.73 100.33 0)
+      (effects (font (size 1.27 1.27)) hide)
+    )
+    (pin "1")
+    (pin "2")
+  )
+  (symbol (lib_id "Resistors_Smd0603:10k") (at 252.73 107.95 90) (unit 1)
+    (in_bom yes) (on_board yes)
+    (property "Reference" "R59" (id 0) (at 265.5316 107.4928 90)
+      (effects (font (size 1.27 1.27)) (justify left))
+    )
+    (property "Value" "10k" (id 1) (at 254.508 108.1278 90)
+      (effects (font (size 1.27 1.27)) (justify left))
+    )
+    (property "Footprint" "Resistor_Smd_0603:10k_0603" (id 2) (at 252.73 107.95 0)
+      (effects (font (size 1.524 1.524)) hide)
+    )
+    (property "Datasheet" "Resistors/Smd_0603/Components_Documentation/Vishay_Resistors_SM0603.pdf" (id 3) (at 252.73 107.95 0)
+      (effects (font (size 1.524 1.524)) hide)
+    )
+    (property "Manufacturer" "ROYAL OHM" (id 4) (at 252.73 107.95 0)
+      (effects (font (size 1.27 1.27)) hide)
+    )
+    (property "Manufacturer Part Number" "0603SAJ0103T5E" (id 5) (at 252.73 107.95 0)
+      (effects (font (size 1.27 1.27)) hide)
+    )
+    (property "Supplier" "TME" (id 6) (at 252.73 107.95 0)
+      (effects (font (size 1.27 1.27)) hide)
+    )
+    (property "Supplier Part Number" "SMD0603-10K" (id 7) (at 252.73 107.95 0)
+      (effects (font (size 1.27 1.27)) hide)
+    )
+    (property "URL" "https://www.tme.eu/pl/details/smd0603-10k/rezystory-smd-0603/royal-ohm/0603saj0103t5e/" (id 8) (at 252.73 107.95 0)
+      (effects (font (size 1.27 1.27)) hide)
+    )
+    (property "Price@1pc" "0,04560" (id 9) (at 252.73 107.95 0)
+      (effects (font (size 1.27 1.27)) hide)
+    )
+    (property "Price@1000pcs" "0,01111" (id 10) (at 252.73 107.95 0)
+      (effects (font (size 1.27 1.27)) hide)
+    )
+    (property "Developer" "MW" (id 11) (at 252.73 107.95 0)
+      (effects (font (size 1.27 1.27)) hide)
+    )
+    (property "Package" "0603" (id 12) (at 252.73 107.95 0)
+      (effects (font (size 1.27 1.27)) hide)
+    )
+    (pin "1")
+    (pin "2")
+  )
   (symbol (lib_id "Resistors_Smd0603:10k") (at 378.46 198.12 0) (unit 1)
     (in_bom yes) (on_board yes)
@@
       (reference "#PWR0199") (unit 1) (value "3V3") (footprint "")
     )
+    (path "/0d1c75e1-d042-4a18-92d9-bcab0bfdf1b5"
+      (reference "#PWR0200") (unit 1) (value "GND") (footprint "")
+    )
     (path "/00000000-0000-0000-0000-000060087a46/00000000-0000-0000-0000-000060123029"
       (reference "#PWR201") (unit 1) (value "3V3") (footprint "")
@@
       (reference "#PWR0207") (unit 1) (value "3V3") (footprint "")
     )
+    (path "/5826c87e-0807-4ae1-868d-0d84f982f0dc"
+      (reference "#PWR0208") (unit 1) (value "GND") (footprint "")
+    )
     (path "/00000000-0000-0000-0000-00005fff457c/00000000-0000-0000-0000-00005ff53261"
       (reference "#PWR0348") (unit 1) (value "GND") (footprint "")
@@
       (reference "R57") (unit 1) (value "220R") (footprint "Resistor_Smd_0603:220R_0603")
     )
+    (path "/618811f1-6b91-4b8e-a4f2-3093c9b8d725"
+      (reference "R58") (unit 1) (value "10k") (footprint "Resistor_Smd_0603:10k_0603")
+    )
+    (path "/3c75bfb3-02ef-4c9f-bb60-965f49fd7b83"
+      (reference "R59") (unit 1) (value "10k") (footprint "Resistor_Smd_0603:10k_0603")
+    )
     (path "/00000000-0000-0000-0000-000060087a46/00000000-0000-0000-0000-000060123023"
       (reference "R60") (unit 1) (value "4k7") (footprint "Resistor_Smd_0603:4k7_0603")
@@
       (reference "TP4") (unit 1) (value "GND") (footprint "Test_Points:Test_Point_2.54mm")
     )
+    (path "/00000000-0000-0000-0000-00005ea691f1/9edb07c6-d72c-496d-8cf4-6cd37c73d522"
+      (reference "TP5") (unit 1) (value "TP1.27mm") (footprint "Test_Points:Test_Point_1.27mm")
+    )
+    (path "/00000000-0000-0000-0000-00005ea691f1/56a90361-b56a-4a96-a810-8a46326e4d59"
+      (reference "TP6") (unit 1) (value "TP1.27mm") (footprint "Test_Points:Test_Point_1.27mm")
+    )
+    (path "/00000000-0000-0000-0000-00005ea691f1/b9866706-c458-4abd-878f-8a9550e15f75"
+      (reference "TP7") (unit 1) (value "TP1.27mm") (footprint "Test_Points:Test_Point_1.27mm")
+    )
+    (path "/00000000-0000-0000-0000-00005ea691f1/a32a7669-965c-4015-be5f-5f21e622a3d6"
+      (reference "TP8") (unit 1) (value "TP1.27mm") (footprint "Test_Points:Test_Point_1.27mm")
+    )
+    (path "/00000000-0000-0000-0000-00005ea691f1/de18ab85-4955-4a1f-8624-386bc2340fbb"
+      (reference "TP9") (unit 1) (value "TP1.27mm") (footprint "Test_Points:Test_Point_1.27mm")
+    )
+    (path "/00000000-0000-0000-0000-00005ea691f1/07482053-3564-44a0-b50c-6fdf3c4349c2"
+      (reference "TP10") (unit 1) (value "TP1.27mm") (footprint "Test_Points:Test_Point_1.27mm")
+    )
+    (path "/00000000-0000-0000-0000-00005ea691f1/31b5e8c4-f9aa-41f6-a5cc-9d536c23e86a"
+      (reference "TP11") (unit 1) (value "TP1.27mm") (footprint "Test_Points:Test_Point_1.27mm")
+    )
     (path "/00000000-0000-0000-0000-00005ea691f1/00000000-0000-0000-0000-00005e88f615/00000000-0000-0000-0000-00005e890c4f"

Commit message: Finalized project, regenerated gerbers
Connections:
- net STM32MP1 module/PD14-GPIO renamed PD14
- net STM32MP1 module/PE14-GPIO renamed PE14
- net STM32MP1 module/PE3-GPIO renamed PE3
- no-connect marks 3 -> 0
Other:
- moved on the sheet: D7, D8, R65, R66

Commit message: Updated schematic
Connections:
- net STLink Module/STM-JTMS-~RESET~ renamed STLink Module/STM-JTMS-~{RESET}
- net STM32MP1 module/STM32-~RST~ renamed STM32MP1 module/STM32-~{RST}
Other:
- sheet MiniPci Module ports: added SPDT_SEL-~{WDISABLE}/UART_RX, ~{RESET}; removed SPDT_SEL-~WDISABLE~/UART_RX, ~RESET~
- sheet STLink Module ports: added STM-JTMS-~{RESET}; removed STM-JTMS-~RESET~
- sheet STM32MP1 module ports: added JTAG-~{TRST}, STM32-~{RST}; removed JTAG-~TRST~, STM32-~RST~
- moved on the sheet: U10
Changed lines of the file:
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@@
-(kicad_sch (version 20210406) (generator eeschema)
+(kicad_sch (version 20210615) (generator eeschema)
   (paper "A3")
   (title_block
@@
       (effects (font (size 1.27 1.27)) (justify left))
     )
-    (pin "~RESET~" input (at 270.51 185.42 180)
+    (pin "~{RESET}" input (at 270.51 185.42 180)
       (effects (font (size 1.27 1.27)) (justify left))
     )
@@
       (effects (font (size 1.27 1.27)) (justify left))
     )
-    (pin "SPDT_SEL-~WDISABLE~{slash}UART_RX" bidirectional (at 270.51 182.88 180)
+    (pin "SPDT_SEL-~{WDISABLE}{slash}UART_RX" bidirectional (at 270.51 182.88 180)
       (effects (font (size 1.27 1.27)) (justify left))
     )
@@
       (effects (font (size 1.27 1.27)) (justify right))
     )
-    (pin "STM-JTMS-~RESET~" input (at 317.5 123.19 0)
+    (pin "STM-JTMS-~{RESET}" input (at 317.5 123.19 0)
       (effects (font (size 1.27 1.27)) (justify right))
     )
@@
       (effects (font (size 1.27 1.27)) (justify right))
     )
-    (pin "STM32-~RST~" input (at 190.5 76.2 180)
+    (pin "STM32-~{RST}" input (at 190.5 76.2 180)
       (effects (font (size 1.27 1.27)) (justify left))
     )
@@
       (effects (font (size 1.27 1.27)) (justify right))
     )
-    (pin "JTAG-~TRST~" input (at 238.76 128.27 0)
-      (effects (font (size 1.27 1.27)) (justify right))
-    )
+    (pin "JTAG-~{TRST}" input (at 238.76 128.27 0)
+      (effects (font (size 1.27 1.27)) (justify right))
+    )
