File: TP_Power_Supply.kicad_sch (KiCad schematic)
At the start: 3 parts, among them U2 MCP1703T-3302E

Commit message: Cleared all errors DRC
Parts:
- C3, C4: symbol Capacitors_Smd0603:1uF_0603 -> Capacitors_Smd0603:1uF; LCSC Part #(optional) (none) -> C105504
Changed lines of the file:
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@@
     (pin "1")
   )
-  (symbol (lib_id "Capacitors_Smd0603:1uF_0603") (at 191.77 147.32 0) (unit 1)
+  (symbol (lib_id "Capacitors_Smd0603:1uF") (at 191.77 147.32 0) (unit 1)
     (in_bom yes) (on_board yes)
     (property "Reference" "C3" (id 0) (at 195.098 146.171 0)
@@
       (effects (font (size 1.524 1.524)) hide)
     )
-    (property "Datasheet" "Capacitors/Smd_0603/Components_Documentation/KEM_C1005_Y5V_SMD.pdf" (id 3) (at 187.96 142.24 0)
+    (property "Datasheet" "https://www.tme.eu/Document/4a42202b32dab16128fe107dd69598cc/samsung-chip-cap.pdf" (id 3) (at 187.96 142.24 0)
       (effects (font (size 1.524 1.524)) hide)
     )
@@
       (effects (font (size 1.27 1.27)) hide)
     )
+    (property "LCSC Part #(optional)" "C105504" (id 12) (at 191.77 147.32 0)
+      (effects (font (size 1.27 1.27)) hide)
+    )
     (pin "1")
     (pin "2")
   )
-  (symbol (lib_id "Capacitors_Smd0603:1uF_0603") (at 232.41 147.32 0) (unit 1)
+  (symbol (lib_id "Capacitors_Smd0603:1uF") (at 232.41 147.32 0) (unit 1)
     (in_bom yes) (on_board yes)
     (property "Reference" "C4" (id 0) (at 235.738 146.171 0)
@@
       (effects (font (size 1.524 1.524)) hide)
     )
-    (property "Datasheet" "Capacitors/Smd_0603/Components_Documentation/KEM_C1005_Y5V_SMD.pdf" (id 3) (at 228.6 142.24 0)
+    (property "Datasheet" "https://www.tme.eu/Document/4a42202b32dab16128fe107dd69598cc/samsung-chip-cap.pdf" (id 3) (at 228.6 142.24 0)
       (effects (font (size 1.524 1.524)) hide)
     )
@@
       (effects (font (size 1.27 1.27)) hide)
     )
+    (property "LCSC Part #(optional)" "C105504" (id 12) (at 232.41 147.32 0)
+      (effects (font (size 1.27 1.27)) hide)
+    )

Commit message: Gerbers created, BOM, CPL
Parts:
- U2: Package SOT-23(SOT-23-3) -> SOT23; Price@1000pcs 1,49 -> 1,52; Price@1pc 2,04 -> 2,09; Supplier TME -> Tme; Supplier Part Number MCP1703T3302ECB -> MCP1703T3302ECB
Changed lines of the file:
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@@
     (pin "1")
   )
+  (symbol (lib_id "Capacitors_Smd0603:1uF") (at 232.41 147.32 0) (unit 1)
+    (in_bom yes) (on_board yes) (fields_autoplaced)
+    (property "Reference" "C4" (id 0) (at 229.0826 146.4115 0)
+      (effects (font (size 1.27 1.27)) (justify right))
+    )
+    (property "Value" "1uF/16V" (id 1) (at 229.0826 149.1866 0)
+      (effects (font (size 1.27 1.27)) (justify right))
+    )
+    (property "Footprint" "Capacitors_Smd_0603:1uF_0603" (id 2) (at 228.6 142.24 0)
+      (effects (font (size 1.524 1.524)) hide)
+    )
+    (property "Datasheet" "https://www.tme.eu/Document/4a42202b32dab16128fe107dd69598cc/samsung-chip-cap.pdf" (id 3) (at 228.6 142.24 0)
+      (effects (font (size 1.524 1.524)) hide)
+    )
+    (property "Manufacturer" "SAMSUNG" (id 4) (at 232.41 147.32 0)
+      (effects (font (size 1.27 1.27)) hide)
+    )
+    (property "Manufacturer Part Number" "CL10B105KO8NNNC" (id 5) (at 232.41 147.32 0)
+      (effects (font (size 1.27 1.27)) hide)
+    )
+    (property "Supplier" "TME" (id 6) (at 232.41 147.32 0)
+      (effects (font (size 1.27 1.27)) hide)
+    )
+    (property "Supplier Part Number" "CL10B105KO8NNNC" (id 7) (at 232.41 147.32 0)
+      (effects (font (size 1.27 1.27)) hide)
+    )
+    (property "URL" "https://www.tme.eu/pl/details/cl10b105ko8nnnc/kondensatory-mlcc-smd-0603/samsung/" (id 8) (at 232.41 147.32 0)
+      (effects (font (size 1.27 1.27)) hide)
+    )
+    (property "Price@1pc" "0,07530" (id 9) (at 232.41 147.32 0)
+      (effects (font (size 1.27 1.27)) hide)
+    )
+    (property "Price@1000pcs" "0,03514" (id 10) (at 232.41 147.32 0)
+      (effects (font (size 1.27 1.27)) hide)
+    )
+    (property "Package" "0603" (id 11) (at 232.41 147.32 0)
+      (effects (font (size 1.27 1.27)) hide)
+    )
+    (property "LCSC Part #(optional)" "C105504" (id 12) (at 232.41 147.32 0)
+      (effects (font (size 1.27 1.27)) hide)
+    )
+    (pin "1")
+    (pin "2")
+  )
   (symbol (lib_id "Capacitors_Smd0603:1uF") (at 191.77 147.32 0) (unit 1)
-    (in_bom yes) (on_board yes)
-    (property "Reference" "C3" (id 0) (at 195.098 146.171 0)
-      (effects (font (size 1.27 1.27)) (justify left))
+    (in_bom yes) (on_board yes) (fields_autoplaced)
+    (property "Reference" "C3" (id 0) (at 188.4426 146.4115 0)
+      (effects (font (size 1.27 1.27)) (justify right))
     )
-    (property "Value" "1uF/16V" (id 1) (at 195.098 148.469 0)
-      (effects (font (size 1.27 1.27)) (justify left))
+    (property "Value" "1uF/16V" (id 1) (at 188.4426 149.1866 0)
+      (effects (font (size 1.27 1.27)) (justify right))
     )
     (property "Footprint" "Capacitors_Smd_0603:1uF_0603" (id 2) (at 187.96 142.24 0)
@@
     (pin "2")
   )
-  (symbol (lib_id "Capacitors_Smd0603:1uF") (at 232.41 147.32 0) (unit 1)
-    (in_bom yes) (on_board yes)
-    (property "Reference" "C4" (id 0) (at 235.738 146.171 0)
-      (effects (font (size 1.27 1.27)) (justify left))
-    )
-    (property "Value" "1uF/16V" (id 1) (at 235.738 148.469 0)
-      (effects (font (size 1.27 1.27)) (justify left))
-    )
-    (property "Footprint" "Capacitors_Smd_0603:1uF_0603" (id 2) (at 228.6 142.24 0)
-      (effects (font (size 1.524 1.524)) hide)
-    )
-    (property "Datasheet" "https://www.tme.eu/Document/4a42202b32dab16128fe107dd69598cc/samsung-chip-cap.pdf" (id 3) (at 228.6 142.24 0)
-      (effects (font (size 1.524 1.524)) hide)
-    )
-    (property "Manufacturer" "SAMSUNG" (id 4) (at 232.41 147.32 0)
-      (effects (font (size 1.27 1.27)) hide)
-    )
-    (property "Manufacturer Part Number" "CL10B105KO8NNNC" (id 5) (at 232.41 147.32 0)
-      (effects (font (size 1.27 1.27)) hide)
-    )
-    (property "Supplier" "TME" (id 6) (at 232.41 147.32 0)
-      (effects (font (size 1.27 1.27)) hide)
-    )
-    (property "Supplier Part Number" "CL10B105KO8NNNC" (id 7) (at 232.41 147.32 0)
-      (effects (font (size 1.27 1.27)) hide)
-    )
-    (property "URL" "https://www.tme.eu/pl/details/cl10b105ko8nnnc/kondensatory-mlcc-smd-0603/samsung/" (id 8) (at 232.41 147.32 0)
-      (effects (font (size 1.27 1.27)) hide)
-    )
-    (property "Price@1pc" "0,07530" (id 9) (at 232.41 147.32 0)
-      (effects (font (size 1.27 1.27)) hide)
-    )
-    (property "Price@1000pcs" "0,03514" (id 10) (at 232.41 147.32 0)
-      (effects (font (size 1.27 1.27)) hide)
-    )
-    (property "Package" "0603" (id 11) (at 232.41 147.32 0)
-      (effects (font (size 1.27 1.27)) hide)
-    )
-    (property "LCSC Part #(optional)" "C105504" (id 12) (at 232.41 147.32 0)
-      (effects (font (size 1.27 1.27)) hide)
-    )
-    (pin "1")
-    (pin "2")
-  )
   (symbol (lib_id "Linear_Regulators:MCP1703T-3302E") (at 212.09 142.24 0) (unit 1)
     (in_bom yes) (on_board yes)
@@
       (effects (font (size 1.524 1.524)) hide)
     )
-    (property "Datasheet" "Dc_Dc_Regulators/Linear/Components_Documentation/Mcp1703T_22049a.pdf" (id 3) (at 212.09 143.51 0)
+    (property "Datasheet" "https://www.tme.eu/Document/de7d38f249f36fadffea0e6430703bcf/_LDO_SG.pdf" (id 3) (at 212.09 143.51 0)
       (effects (font (size 1.524 1.524)) hide)
     )
@@
       (effects (font (size 1.27 1.27)) hide)
     )
-    (property "Supplier" "TME" (id 6) (at 212.09 142.24 0)
+    (property "Supplier" "Tme" (id 6) (at 212.09 142.24 0)
       (effects (font (size 1.27 1.27)) hide)
     )
-    (property "Supplier Part Number" "MCP1703T3302ECB" (id 7) (at 212.09 142.24 0)
+    (property "Supplier Part Number" "MCP1703T3302ECB " (id 7) (at 212.09 142.24 0)
       (effects (font (size 1.27 1.27)) hide)
     )
@@
       (effects (font (size 1.27 1.27)) hide)
     )
-    (property "Price@1pc" "2,04" (id 9) (at 212.09 142.24 0)
+    (property "Price@1pc" "2,09" (id 9) (at 212.09 142.24 0)
       (effects (font (size 1.27 1.27)) hide)
     )
-    (property "Price@1000pcs" "1,49" (id 10) (at 212.09 142.24 0)
+    (property "Price@1000pcs" "1,52" (id 10) (at 212.09 142.24 0)
       (effects (font (size 1.27 1.27)) hide)
     )
@@
       (effects (font (size 1.27 1.27)) hide)
     )
-    (property "Package" "SOT-23(SOT-23-3)" (id 12) (at 212.09 142.24 0)
+    (property "Package" "SOT23" (id 12) (at 212.09 142.24 0)
       (effects (font (size 1.27 1.27)) hide)
     )
